File: Тестовые драйвера.kicad_sch (KiCad schematic)
At the start: 136 parts, among them J1 Conn_02x10_Odd_Even, J2 Conn_02x10_Odd_Even, J3 Conn_01x01, J4 Conn_01x01, Q1 C2M0280120D, Q2 C2M0280120D, Q3 C2M0280120D, Q4 C2M0280120D, Q5 C2M0280120D, Q6 C2M0280120D

Commit message: Полная схема
Parts:
- removed C59, C62: CY, Capacitor_SMD:C_0603_1608Metric_Pad1.08x0.95mm_HandSolder, symbol Device:C_Small
- removed R6: 0, Resistor_SMD:R_0805_2012Metric_Pad1.20x1.40mm_HandSolder, symbol Device:R_Small
- added C60, C61: 4.7u, Capacitor_SMD:C_0603_1608Metric_Pad1.08x0.95mm_HandSolder, symbol Device:C_Small
- added C61: 10u, Capacitor_SMD:C_0603_1608Metric_Pad1.08x0.95mm_HandSolder, symbol Device:C_Small
- added C62 (x3): CY-270p, Capacitor_SMD:C_0603_1608Metric_Pad1.08x0.95mm_HandSolder, symbol Device:C_Small
- added C9 (x9): 56p, Capacitor_SMD:C_0603_1608Metric_Pad1.08x0.95mm_HandSolder, symbol Device:C_Small
- added C9 (x3): 1u, Capacitor_SMD:C_0603_1608Metric_Pad1.08x0.95mm_HandSolder, symbol Device:C_Small
- added J1, J2, J3: Conn_01x01, Connector_My:Power_Wire, symbol Connector_Generic:Conn_01x01
- added L2: 6.8u, Inductor_SMD:L_1812_4532Metric_Pad1.30x3.40mm_HandSolder, symbol Device:L_Small
- added PS3: B1203S-1WR3, Converter_DCDC:Converter_DCDC_RECOM_R-78S-0.1_THT, symbol Converter_DCDC:IA1203S
- added R5 (x9): 120, Resistor_SMD:R_0805_2012Metric_Pad1.20x1.40mm_HandSolder, symbol Device:R_Small
- added R6 (x4): 0, Resistor_SMD:R_0805_2012Metric_Pad1.20x1.40mm_HandSolder, symbol Device:R_Small
- added U1, U2, U3: 74AHC1G08, Package_SO:TSOP-5_1.65x3.05mm_P0.95mm, symbol 74xGxx:74AHC1G08
- D6, D7: footprint (none) -> LED_SMD:LED_0805_2012Metric_Pad1.15x1.40mm_HandSolder
- PS1, PS2: value IA1215S -> A1215S-1WR3
- renumbered J3 to J4, J4 to J5, J1 to J6, J2 to J7
Connections:
- net +12V: now also C60.1, L2.1
- net +3.3V: now also C61.1, C9.1, C9.1, C9.1, PS3.4 (+Vout), U1.5 (VCC), U2.5 (VCC), U3.5 (VCC)
- net GND: now also C61.2, C62.2, C9.2, C9.2, C9.2, C9.2, C9.2, C9.2, C9.2, C9.2, C9.2, C9.2, C9.2, C9.2, PS3.3 (0V), U1.3 (GND), U2.3 (GND), U3.3 (GND); no longer C55.2, C56.2, C60.2, C61.2, PS1.2 (-Vin), PS2.2 (-Vin)
- net GND2H: now also C62.2, J2.1 (Pin_1)
- net GNDPWR: now also C62.2, J1.1 (Pin_1)
- net IN+H: now also R6.1, R6.2
- net IN+L: now also R6.2, R6.2
- net IN-H: now also R6.1
- net IN-L: now also R6.2
- net RDYH: now also R5.2
- net RDYL: now also R5.2
- net VDC: now also J3.1 (Pin_1)
- net ~{FLTH}: now also R5.2
- net ~{FLTL}: now also R5.2
- net ~{RSTH}: now also R6.1
- net ~{RSTL}: now also R6.1
- net HighERR: now reaches J7.13 (Pin_13)
- net HighERR: now also J6.13 (Pin_13), C9.1, R5.1, R5.2
- net LowERR: now reaches J7.15 (Pin_15)
- net LowERR: now also J6.15 (Pin_15), C9.1, R5.1, R5.2
- net CommonERR: now reaches J7.17 (Pin_17)
- net CommonERR: now also J6.17 (Pin_17), C9.1, R5.1
- new net: C9.1, R5.1, U3.2
- new net: R5.2, U2.4
- new net: C9.1, R5.1, U2.2
- new net: C9.1, R5.1, U2.1
- new net: C61.1, L2.2, PS3.2 (+Vin)
- new net: C9.1, R5.1, U3.1
- new net: R5.2, U3.4
- new net: C9.1, R5.1, U1.2
- new net: C9.1, R5.1, U1.1
- new net: R5.2, U1.4
- new net GND1: C55.2, C56.2, C60.2, C60.2, C61.2, C61.2, C62.1, C62.1, C62.1, PS1.2 (-Vin), PS2.2 (-Vin), PS3.1 (-Vin)
Other:
- note added: "Автоматический RST"
- note added: "Защита от одновременного включения"
- note added: "Общая ошибка"
- note added: "Опции ERROR"
- note added: "Опции RESET"
- note added: "Ошибка верхнего драйвера"
- note added: "Ошибка нижнего драйвера"
- note added: "Питание 3.3В опционально"
- note added: "Разъёмы питания"
- note added: "Силовые разъёмы"
- note removed: "Перемычка RESET"
- moved on the sheet: J4, J5, J6, J7
