File: Тестовые драйвера.kicad_pcb (KiCad board)
At the start: 2 copper layers, 135 parts, among them J1 Conn_02x10_Odd_Even, J2 Conn_02x10_Odd_Even, J3 Conn_01x01, J4 Conn_01x01, Q1 C2M0280120D, Q2 C2M0280120D, Q3 C2M0280120D, Q4 C2M0280120D, Q5 C2M0280120D, Q6 C2M0280120D

Commit message: Полная схема
Parts:
- added C41: 100n, Capacitor_SMD:C_0603_1608Metric_Pad1.08x0.95mm_HandSolder, F.Cu at (179.4, 30.4)
- added C42: Cf, Capacitor_SMD:C_0603_1608Metric_Pad1.08x0.95mm_HandSolder, F.Cu at (179.4, 32.9)
- added C43: 1u, Capacitor_SMD:C_0603_1608Metric_Pad1.08x0.95mm_HandSolder, F.Cu at (179.4, 35.4)
- added C44: 1u, Capacitor_SMD:C_0603_1608Metric_Pad1.08x0.95mm_HandSolder, F.Cu at (179.4, 37.9)
- added C45: 1u, Capacitor_SMD:C_0603_1608Metric_Pad1.08x0.95mm_HandSolder, F.Cu at (183.8, 30.4)
- added C46: 56p, Capacitor_SMD:C_0603_1608Metric_Pad1.08x0.95mm_HandSolder, F.Cu at (183.8, 32.9)
- added C47: 56p, Capacitor_SMD:C_0603_1608Metric_Pad1.08x0.95mm_HandSolder, F.Cu at (183.8, 35.4)
- added C48: 56p, Capacitor_SMD:C_0603_1608Metric_Pad1.08x0.95mm_HandSolder, F.Cu at (183.8, 37.9)
- added C49: 56p, Capacitor_SMD:C_0603_1608Metric_Pad1.08x0.95mm_HandSolder, F.Cu at (188.1, 30.4)
- added C50: 56p, Capacitor_SMD:C_0603_1608Metric_Pad1.08x0.95mm_HandSolder, F.Cu at (188.1, 32.9)
- added C51: 56p, Capacitor_SMD:C_0603_1608Metric_Pad1.08x0.95mm_HandSolder, F.Cu at (188.1, 35.4)
- added C52: 56p, Capacitor_SMD:C_0603_1608Metric_Pad1.08x0.95mm_HandSolder, F.Cu at (188.1, 37.9)
- added C53: 56p, Capacitor_SMD:C_0603_1608Metric_Pad1.08x0.95mm_HandSolder, F.Cu at (86.6, 74.7)
- added C54: 56p, Capacitor_SMD:C_0603_1608Metric_Pad1.08x0.95mm_HandSolder, F.Cu at (86.6, 77.2)
- added C55: 100n, Capacitor_SMD:C_0603_1608Metric_Pad1.08x0.95mm_HandSolder, F.Cu at (86.6, 79.7)
- added C56: Cf, Capacitor_SMD:C_0603_1608Metric_Pad1.08x0.95mm_HandSolder, F.Cu at (86.6, 82.2)
- added D7: LED_Small, LED_SMD:LED_0805_2012Metric_Pad1.15x1.40mm_HandSolder, F.Cu at (173.2, 107.2)
- added J5: Conn_01x01, Connector_My:Power_Wire, F.Cu at (81.4, 76.4)
- added J6: Conn_02x10_Odd_Even, Connector_PinSocket_2.54mm:PinSocket_2x10_P2.54mm_Vertical, F.Cu at (81.4, 82.4)
- added J7: Conn_02x10_Odd_Even, Connector_PinHeader_2.54mm:PinHeader_2x10_P2.54mm_Vertical, F.Cu at (73.5, 75.8)
- added L3: 6.8u, Inductor_SMD:L_1812_4532Metric_Pad1.30x3.40mm_HandSolder, F.Cu at (82.1, 98.0)
- added PS3: B1203S-1WR3, Converter_DCDC:Converter_DCDC_RECOM_R-78S-0.1_THT, F.Cu at (81.3, 92.7)
- added R44: 120, Resistor_SMD:R_0805_2012Metric_Pad1.20x1.40mm_HandSolder, F.Cu at (168.9, 26.0)
- added R45: 120, Resistor_SMD:R_0805_2012Metric_Pad1.20x1.40mm_HandSolder, F.Cu at (168.9, 28.9)
- added R46: 120, Resistor_SMD:R_0805_2012Metric_Pad1.20x1.40mm_HandSolder, F.Cu at (168.9, 31.9)
- added R47: 120, Resistor_SMD:R_0805_2012Metric_Pad1.20x1.40mm_HandSolder, F.Cu at (168.9, 34.8)
- added R48: 120, Resistor_SMD:R_0805_2012Metric_Pad1.20x1.40mm_HandSolder, F.Cu at (168.9, 37.8)
- added R49: 120, Resistor_SMD:R_0805_2012Metric_Pad1.20x1.40mm_HandSolder, F.Cu at (168.9, 40.7)
- added R50: 120, Resistor_SMD:R_0805_2012Metric_Pad1.20x1.40mm_HandSolder, F.Cu at (168.9, 43.7)
- added R51: 15, Resistor_SMD:R_1206_3216Metric_Pad1.30x1.75mm_HandSolder, F.Cu at (174.3, 30.8)
- added R52: 15, Resistor_SMD:R_1206_3216Metric_Pad1.30x1.75mm_HandSolder, F.Cu at (174.3, 34.0)
- added R53: 15, Resistor_SMD:R_1206_3216Metric_Pad1.30x1.75mm_HandSolder, F.Cu at (174.3, 37.3)
- added R54: 15, Resistor_SMD:R_1206_3216Metric_Pad1.30x1.75mm_HandSolder, F.Cu at (174.3, 40.6)
- added R55: Rdesat, Resistor_SMD:R_0805_2012Metric_Pad1.20x1.40mm_HandSolder, F.Cu at (168.9, 46.6)
- added U1: 74AHC1G08, Package_SO:TSOP-5_1.65x3.05mm_P0.95mm, F.Cu at (173.6, 26.8)
- added U2: 74AHC1G08, Package_SO:TSOP-5_1.65x3.05mm_P0.95mm, F.Cu at (178.1, 26.8)
- added U3: 74AHC1G08, Package_SO:TSOP-5_1.65x3.05mm_P0.95mm, F.Cu at (182.7, 26.8)
- C23, C9: value CY -> CY-270p
- C24: value 10u -> 4.7u
- C25: value 0.1u -> 4.7u
- C26, C37: value 100n -> 10u
- C27: value Cf -> 10u
- C29: value 1u -> 100n
- C30: value Cblk -> Cf
- C31: value 0.1n -> CY-270p
- C32: value 0.1n -> 0.1u
- C33: value 10u -> 1u
- C34: value 0.1u -> Cblk
- C35: value 100n -> 0.1n
- C36: value Cf -> 0.1n
- C38: value Cf -> 0.1u
- D6: value D_Small -> LED_Small; footprint Diode_SMD:D_SMA_Handsoldering -> LED_SMD:LED_0805_2012Metric_Pad1.15x1.40mm_HandSolder
- J1: value Conn_02x10_Odd_Even -> Conn_01x01; footprint Connector_PinSocket_2.54mm:PinSocket_2x10_P2.54mm_Vertical -> Connector_My:Power_Wire
- J2: value Conn_02x10_Odd_Even -> Conn_01x01; footprint Connector_PinHeader_2.54mm:PinHeader_2x10_P2.54mm_Vertical -> Connector_My:Power_Wire
- PS1, PS2: value IA1215S -> A1215S-1WR3
- R26: value 0 -> 330
- R28: value 330 -> 0
- R29, R30, R31: value 15 -> 0; footprint Resistor_SMD:R_1206_3216Metric_Pad1.30x1.75mm_HandSolder -> Resistor_SMD:R_0805_2012Metric_Pad1.20x1.40mm_HandSolder
- R33, R38: value Rdesat -> 15; footprint Resistor_SMD:R_0805_2012Metric_Pad1.20x1.40mm_HandSolder -> Resistor_SMD:R_1206_3216Metric_Pad1.30x1.75mm_HandSolder
- R36, R41: value 15 -> Rdesat; footprint Resistor_SMD:R_1206_3216Metric_Pad1.30x1.75mm_HandSolder -> Resistor_SMD:R_0805_2012Metric_Pad1.20x1.40mm_HandSolder
- R42: value 15 -> 120; footprint Resistor_SMD:R_1206_3216Metric_Pad1.30x1.75mm_HandSolder -> Resistor_SMD:R_0805_2012Metric_Pad1.20x1.40mm_HandSolder
- R43: value Rdesat -> 120
- moved D8 119.5 mm to (65.6, 137.8)
Connections:
- C18 pad 2: GND -> GND1
- C19 pad 2: GND -> GND1
- C23 pad 1: GND -> GND1
- C24 pad 1: GNDPWR -> +12V
- C24 pad 2: +15VH -> GND1
- C25 pad 1: GNDPWR -> Net-(PS3-+Vin)
- C25 pad 2: +15VH -> GND1
- C26 pad 1: ClampH -> +3.3V
- C26 pad 2: OUT -> GND
- C27 pad 1: Net-(C27-Pad1) -> GNDPWR
- C27 pad 2: OUT -> +15VH
- C28 pad 1: GND -> GNDPWR
- C28 pad 2: +3.3V -> +15VH
- C29 pad 1: GND -> ClampH
- C29 pad 2: +3.3V -> OUT
- C30 pad 1: GNDPWR -> Net-(C30-Pad1)
- C30 pad 2: Net-(D8-DESAT) -> OUT
- C31 pad 1: ~{FLTL} -> GND1
- C32 pad 1: RDYL -> GND
- C32 pad 2: GND -> +3.3V
- C33 pad 1: +15VH -> GND
- C33 pad 2: GNDPWR -> +3.3V
- C34 pad 1: +15VH -> GNDPWR
- C34 pad 2: GNDPWR -> Net-(D8-DESAT)
- C35 pad 1: ClampL -> ~{FLTL}
- C35 pad 2: GNDPWR -> GND
- C36 pad 1: Net-(C36-Pad1) -> RDYL
- C36 pad 2: GNDPWR -> GND
- C37 pad 1: ClampL -> +15VH
- C38 pad 1: Net-(C38-Pad1) -> +15VH
- C4 pad 2: GND -> GND1
- C5 pad 2: GND -> GND1
- C9 pad 1: GND -> GND1
- D6 pad 1: Net-(D5-A) -> GND
- D6 pad 2: Net-(D13-A) -> Net-(D6-A)
- J1 pad 1: +3.3V -> GNDPWR
- J2 pad 1: +3.3V -> OUT
- J3 pad 1: GND -> VDC
- J4 pad 1: +12V -> GND
- PS1 pad 2: GND -> GND1
- PS2 pad 2: GND -> GND1
- R21 pad 1: Net-(C27-Pad1) -> Net-(C30-Pad1)
- R26 pad 1: ~{RSTL} -> RDYL
- R26 pad 2: ~{RSTH} -> Net-(D13-A)
- R27 pad 1: RDYL -> ~{FLTL}
- R27 pad 2: Net-(D13-A) -> Net-(D14-K)
- R28 pad 1: ~{FLTL} -> IN+H
- R28 pad 2: Net-(D14-K) -> IN-L
- R29 pad 1: OutH2 -> IN-H
- R29 pad 2: Net-(R29-Pad2) -> IN+L
- R30 pad 1: Net-(R29-Pad2) -> ~{RSTL}
- R30 pad 2: ClampL -> IN+L
- R31 pad 1: Net-(R31-Pad1) -> ~{RSTH}
- R31 pad 2: OutL2 -> IN+H
- R32 pad 1: ClampL -> OutH2
- R32 pad 2: Net-(R31-Pad1) -> Net-(R32-Pad2)
- R33 pad 1: Net-(C36-Pad1) -> Net-(R32-Pad2)
- R34 pad 1: OutH2 -> Net-(R34-Pad1)
- R34 pad 2: Net-(R34-Pad2) -> OutL2
- R35 pad 1: Net-(R34-Pad2) -> ClampL
- R35 pad 2: ClampL -> Net-(R34-Pad1)
- R36 pad 1: Net-(R36-Pad1) -> Net-(C40-Pad1)
- R36 pad 2: OutL2 -> ClampL
- R37 pad 1: ClampL -> OutH2
- R37 pad 2: Net-(R36-Pad1) -> Net-(R37-Pad2)
- R38 pad 1: Net-(C38-Pad1) -> Net-(R37-Pad2)
- R39 pad 1: OutH2 -> Net-(R39-Pad1)
- R39 pad 2: Net-(R39-Pad2) -> OutL2
- R40 pad 1: Net-(R39-Pad2) -> ClampL
- R40 pad 2: ClampL -> Net-(R39-Pad1)
- R41 pad 1: Net-(R41-Pad1) -> Net-(C42-Pad1)
- R41 pad 2: OutL2 -> ClampL
- R42 pad 1: ClampL -> Net-(C46-Pad1)
- R42 pad 2: Net-(R41-Pad1) -> RDYH
- R43 pad 1: Net-(C40-Pad1) -> Net-(C47-Pad1)
- R43 pad 2: ClampL -> RDYL

Commit message: Начал разводку платы
Parts:
- C1, C23, C4, C5, C6, C9: footprint Capacitor_SMD:C_0603_1608Metric_Pad1.08x0.95mm_HandSolder -> Capacitor_SMD:C_1210_3225Metric_Pad1.33x2.70mm_HandSolder
- C12, C13, C14, C16, C17, C2, C3, C32, C33, C34, C7, C8: footprint Capacitor_SMD:C_0603_1608Metric_Pad1.08x0.95mm_HandSolder -> Capacitor_SMD:C_0805_2012Metric_Pad1.18x1.45mm_HandSolder
- C15, C18, C19, C20: footprint Capacitor_SMD:C_0603_1608Metric_Pad1.08x0.95mm_HandSolder -> Capacitor_SMD:C_1210_3225Metric_Pad1.33x2.70mm_HandSolder; moved to B.Cu
- C27, C28, C35, C36, C37, C38: footprint Capacitor_SMD:C_0603_1608Metric_Pad1.08x0.95mm_HandSolder -> Capacitor_SMD:C_0805_2012Metric_Pad1.18x1.45mm_HandSolder; moved to B.Cu
- L2, R24, R25: moved to B.Cu
- moved TP5 175.6 mm to (119.4, 217.6)
- moved TP6 174.9 mm to (119.4, 221.4)
- moved R51 169.9 mm to (90.2, 178.4)
- moved R53 166.4 mm to (90.2, 181.0), turned to 180 degrees
- moved R23 162.5 mm to (94.0, 164.5)
- moved R32 162.0 mm to (90.2, 168.3)
- moved D12 157.1 mm to (81.9, 164.5), turned to 180 degrees
- moved D11 155.8 mm to (71.1, 164.5), turned to 180 degrees
- moved R39 155.6 mm to (90.2, 175.9), turned to 180 degrees
- moved R26 144.3 mm to (123.2, 170.2)
- moved D9 141.7 mm to (51.4, 164.5)
- moved R34 140.6 mm to (90.2, 170.8), turned to 180 degrees
- moved R37 137.7 mm to (90.2, 173.4)
- moved R22 134.7 mm to (89.5, 164.5)
- moved C38 132.1 mm to (97.2, 175.9), turned to 180 degrees
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Connections:
- C15 pad 1: +15VH -> +15VL
- C16 pad 1: +15VH -> -15VH
- C17 pad 1: +15VH -> -15VH
- C20 pad 2: +15VH -> -15VL
- C27 pad 2: +15VH -> +15VL
- C28 pad 2: +15VH -> +15VL
- C37 pad 1: +15VH -> -15VL
- C38 pad 1: +15VH -> -15VL
- C6 pad 2: +15VH -> -15VH
- D1 pad 1: +15VH -> -15VH
- D1 pad 8: +15VH -> -15VH
- D8 pad 1: +15VH -> -15VL
- D8 pad 5: +15VH -> +15VL
- D8 pad 8: +15VH -> -15VL
- PS1 pad 4: +15VH -> -15VH
- PS2 pad 4: +15VH -> -15VL
- PS2 pad 6: +15VH -> +15VL
Routing:
- net RDYL: track 0.00 -> 17.5 mm, vias 0 -> 1
- net ~{FLTL}: track 0.00 -> 16.4 mm, vias 0 -> 1
- net GNDPWR: track 0.00 -> 8.78 mm, vias 0 -> 1
- net GND: track 0.00 -> 8.48 mm
- net Net-(D8-DESAT): track 0.00 -> 6.90 mm
- net +15VL: track 0.00 -> 6.24 mm, vias 0 -> 1
- net -15VL: track 0.00 -> 5.74 mm, vias 0 -> 1
- net +3.3V: track 0.00 -> 5.61 mm
- net ~{RSTL}: track 0.00 -> 2.34 mm, vias 0 -> 1
- net Net-(D14-K): track 0.00 -> 1.78 mm
- net Net-(D13-A): track 0.00 -> 1.78 mm

Commit message: Расположил на плате
Parts:
- C1, C13, C14, C16, C17, C2, C3, C4, C5, C6, L1, R16, R21, R36, R41, R5, R55, R8, R9: moved to B.Cu
- C10, C11, C21, C22, C29, C30, C39, C40, C41, C42, C55, C56: footprint Capacitor_SMD:C_0603_1608Metric_Pad1.08x0.95mm_HandSolder -> Capacitor_SMD:C_0805_2012Metric_Pad1.18x1.45mm_HandSolder; moved to B.Cu
- moved C53 178.1 mm to (263.2, 97.4)
- moved C54 178.1 mm to (263.2, 99.9)
- moved PS3 178.1 mm to (257.9, 115.4)
- moved J5 178.1 mm to (258.1, 99.1)
- moved J6 178.1 mm to (258.1, 105.1)
- moved J7 178.1 mm to (250.2, 98.4)
- moved L3 178.1 mm to (258.7, 120.7)
- moved R35 157.3 mm to (66.7, 121.3)
- moved R52 151.2 mm to (66.7, 140.3), turned to 180 degrees
- moved R16 149.4 mm to (63.5, 95.5), turned to -90 degrees
- moved R13 148.9 mm to (66.7, 97.2), turned to 180 degrees
- moved R20 148.5 mm to (66.7, 110.5)
- moved R54 148.4 mm to (66.7, 142.9)
- moved R15 148.0 mm to (66.7, 99.7)
- moved C41 148.0 mm to (66.0, 125.5), turned to 90 degrees
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Routing:
- net Net-(D1-DESAT): track 0.00 -> 7.40 mm
- net GNDPWR: track 8.78 -> 12.4 mm, vias 1 -> 2
- net Net-(D8-DESAT): track 6.90 -> 10.2 mm
- net Net-(R22-Pad2): track 0.00 -> 2.45 mm
- net OUT: track 0.00 -> 1.70 mm, vias 0 -> 1
- net ClampL: track 0.00 -> 1.70 mm, vias 0 -> 1
- net -15VH: track 0.00 -> 1.70 mm, vias 0 -> 1
- net +15VH: track 0.00 -> 1.70 mm, vias 0 -> 1
- net ~{RSTH}: vias 0 -> 1
- net ~{FLTH}: vias 0 -> 1
- net RDYH: vias 0 -> 1
- added copper zone on F.Cu, net OutH2
- added copper zone on F.Cu, net OutL2

Commit message: Разве драйвера
Parts:
- moved R17 5.08 mm to (79.4, 94.6)
- moved R1 2.54 mm to (79.4, 89.5)
- moved R12 2.54 mm to (79.4, 92.1)
- moved R14 2.54 mm to (79.4, 99.7)
- moved R3 2.54 mm to (79.4, 97.2)
- turned C13 to 0 degrees
- turned C14 to 0 degrees
- turned C6 to 0 degrees
- turned C9 to 180 degrees
- turned D6 to 180 degrees
- turned R8 to 0 degrees
- turned R9 to 0 degrees
Routing:
- net ClampH: track 0.00 -> 125.0 mm, vias 0 -> 1
- net ClampL: track 1.70 -> 123.8 mm
- net OUT: track 1.70 -> 68.8 mm, vias 1 -> 4
- net VDC: track 0.00 -> 33.6 mm, vias 0 -> 1
- net GND1: track 0.00 -> 30.7 mm
- net GNDPWR: track 12.4 -> 37.8 mm, vias 2 -> 4
- net Net-(D12-K): track 0.00 -> 25.2 mm, vias 0 -> 2
- net RDYH: track 0.00 -> 17.5 mm
- net ~{FLTH}: track 0.00 -> 16.4 mm
- net -15VH: track 1.70 -> 14.6 mm, vias 1 -> 4
- net +3.3V: track 5.61 -> 16.2 mm, vias 0 -> 4
- net -15VL: track 5.74 -> 14.9 mm, vias 1 -> 4
- net GND: track 8.48 -> 17.0 mm
- net +15VH: track 1.70 -> 9.74 mm
- net Net-(D4-K): track 0.00 -> 7.80 mm
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- added copper zone on B.Cu, net +15VH
- added copper zone on B.Cu, net +15VL
- added copper zone on In2.Cu, net -15VH
- added copper zone on In2.Cu, net -15VL
- added copper zone on B.Cu, net GNDPWR
- added copper zone on F.Cu, net Net-(R1-Pad2)
- added copper zone on B.Cu, net Net-(R12-Pad2)
- added copper zone on F.Cu, net Net-(R14-Pad1)
- added copper zone on B.Cu, net Net-(R17-Pad2)
- added copper zone on F.Cu, net Net-(R19-Pad1)
- added copper zone on F.Cu, net Net-(R3-Pad1)
- added copper zone on F.Cu, net Net-(R32-Pad2)
- added copper zone on F.Cu, net Net-(R34-Pad1)
- added copper zone on B.Cu, net Net-(R37-Pad2)
- added copper zone on F.Cu, net Net-(R39-Pad1)
- added copper zone on B.Cu, net Net-(R51-Pad2)
- added copper zone on F.Cu, net Net-(R53-Pad1)
- added copper zone on B.Cu, net OUT
- added copper zone on F.Cu, net OutH1
- added copper zone on F.Cu, net OutL1
Other:
- copper layers 2 -> 4

Commit message: Закончил схему и разводку платы
Parts:
- removed C44, C45: 1u, Capacitor_SMD:C_0603_1608Metric_Pad1.08x0.95mm_HandSolder
- removed C48, C51, C54: 56p, Capacitor_SMD:C_0603_1608Metric_Pad1.08x0.95mm_HandSolder
- removed J7: Conn_02x10_Odd_Even, Connector_PinHeader_2.54mm:PinHeader_2x10_P2.54mm_Vertical
- removed U1, U2: 74AHC1G08, Package_SO:TSOP-5_1.65x3.05mm_P0.95mm
- added D15: MBR0520, Diode_My:D_SOD_123_Hand, F.Cu at (130.2, 120.0)
- added D16: MBR0520, Diode_My:D_SOD_123_Hand, F.Cu at (132.0, 95.9)
- added R56: 0.5m, Shunt_My:LR2725, F.Cu at (47.0, 114.9)
- added R57: 0.5m, Shunt_My:LR2725, F.Cu at (47.0, 104.1)
- added R58: 1k, Resistor_SMD:R_0805_2012Metric_Pad1.20x1.40mm_HandSolder, F.Cu at (136.9, 98.4)
- added TP26: TestPoint, TestPoint:TestPoint_Loop_D2.50mm_Drill1.0mm_LowProfile, F.Cu at (74.9, 118.1)
- C24, C25: footprint Capacitor_SMD:C_0603_1608Metric_Pad1.08x0.95mm_HandSolder -> Capacitor_SMD:C_1210_3225Metric_Pad1.33x2.70mm_HandSolder
- C26, C31: footprint Capacitor_SMD:C_0603_1608Metric_Pad1.08x0.95mm_HandSolder -> Capacitor_SMD:C_1210_3225Metric_Pad1.33x2.70mm_HandSolder; moved to B.Cu
- C43: footprint Capacitor_SMD:C_0603_1608Metric_Pad1.08x0.95mm_HandSolder -> Capacitor_SMD:C_0805_2012Metric_Pad1.18x1.45mm_HandSolder; moved to B.Cu
- C46, C47, C49, C50, C52, C53: footprint Capacitor_SMD:C_0603_1608Metric_Pad1.08x0.95mm_HandSolder -> Capacitor_SMD:C_0805_2012Metric_Pad1.18x1.45mm_HandSolder
- J1, J2, J3: footprint Connector_My:Power_Wire -> Connector_Power_My:Cuprum_M4
- R47: value 120 -> 2k
- U3: value 74AHC1G08 -> HEF4082BT; footprint Package_SO:TSOP-5_1.65x3.05mm_P0.95mm -> Package_SO:SO-14_3.9x8.65mm_P1.27mm
- moved J3 218.1 mm to (25.4, 83.1)
- moved J1 216.8 mm to (25.4, 136.5)
- moved J2 214.2 mm to (25.4, 109.5)
- moved TP7 147.6 mm to (74.9, 85.7)
- moved J5 139.0 mm to (121.3, 74.3)
- moved PS3 135.7 mm to (127.3, 78.4)
- moved C53 133.7 mm to (130.1, 109.2)
- moved C24 133.6 mm to (128.6, 87.0), turned to 180 degrees
- moved C25 133.3 mm to (128.6, 82.5), turned to 180 degrees
- moved L3 130.2 mm to (133.6, 84.5), turned to 90 degrees
- moved J4 128.6 mm to (114.3, 74.3)
- moved C26 128.4 mm to (133.6, 74.9), turned to 180 degrees
- moved J6 114.1 mm to (144.2, 97.8)
- moved R29 112.2 mm to (111.1, 105.1), turned to -90 degrees
- moved R30 110.2 mm to (102.2, 129.5), turned to 90 degrees
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Connections:
- C1 pad 2: OUT -> GND2H
- C10 pad 2: OUT -> GND2H
- C11 pad 2: OUT -> GND2H
- C12 pad 1: OUT -> GND2H
- C16 pad 2: OUT -> GND2H
- C17 pad 2: OUT -> GND2H
- C2 pad 1: OUT -> GND2H
- C21 pad 2: OUT -> GND2H
- C22 pad 2: OUT -> GND2H
- C29 pad 2: OUT -> GND2H
- C3 pad 1: OUT -> GND2H
- C30 pad 2: OUT -> GND2H
- C46 pad 1: Net-(C46-Pad1) -> Net-(U3-1A)
- C47 pad 1: Net-(C47-Pad1) -> Net-(U3-2A)
- C50 pad 1: LowERR -> GND
- C50 pad 2: GND -> LowERR
- C52 pad 1: Net-(C52-Pad1) -> Net-(U3-1B)
- C53 pad 1: Net-(C53-Pad1) -> Net-(U3-2B)
- C6 pad 1: OUT -> GND2H
- C9 pad 2: OUT -> GND2H
- D1 pad 3: OUT -> GND2H
- D9 pad 1: OUT -> Drain_Low
- J4 pad 1: GND -> GND1
- J6 pad 10: RDYL -> HighERR
- J6 pad 11: ~{FLTH} -> GND
- J6 pad 12: ~{FLTL} -> LowERR_ADC
- J6 pad 13: HighERR -> GND
- J6 pad 14: unconnected-(J6-Pin_14-Pad14) -> HighERR_ADC
- J6 pad 15: LowERR -> GND
- J6 pad 16: unconnected-(J6-Pin_16-Pad16) -> IN+L
- J6 pad 17: CommonERR -> GND
- J6 pad 18: unconnected-(J6-Pin_18-Pad18) -> IN-L
- J6 pad 19: unconnected-(J6-Pin_19-Pad19) -> GND
- J6 pad 2: GND -> ~{RSTH}
- J6 pad 20: unconnected-(J6-Pin_20-Pad20) -> ~{RSTL}
- J6 pad 3: ~{RSTH} -> +3.3V
- J6 pad 4: ~{RSTL} -> IN+H
- J6 pad 5: IN+H -> +3.3V
- J6 pad 6: IN+L -> IN-H
- J6 pad 7: IN-H -> +3.3V
- J6 pad 8: IN-L -> LowERR
- J6 pad 9: RDYH -> +3.3V
- PS1 pad 5: OUT -> GND2H
- Q1 pad 3: OUT -> GND2H
- Q2 pad 3: OUT -> GND2H
- Q3 pad 3: OUT -> GND2H
- Q4 pad 2: OUT -> Drain_Low
- Q5 pad 2: OUT -> Drain_Low
- Q6 pad 2: OUT -> Drain_Low
- R42 pad 1: Net-(C46-Pad1) -> Net-(U3-1A)
- R43 pad 1: Net-(C47-Pad1) -> Net-(U3-2A)
- R44 pad 1: Net-(C48-Pad1) -> Net-(D15-K)
- R44 pad 2: HighERR -> HighERR_ADC
- R45 pad 2: Net-(R45-Pad2) -> Net-(U3-1Y)
- R46 pad 2: Net-(R46-Pad2) -> Net-(U3-2Y)
- R47 pad 1: CommonERR -> GND
- R47 pad 2: Net-(R47-Pad2) -> HighERR_ADC
- R48 pad 1: Net-(C52-Pad1) -> Net-(U3-1B)
- R49 pad 1: Net-(C53-Pad1) -> Net-(U3-2B)
- R50 pad 1: Net-(C54-Pad1) -> Net-(D16-K)
- R50 pad 2: LowERR -> LowERR_ADC
- TP10 pad 1: OUT -> GND2H
- TP13 pad 1: OUT -> GND2H
- TP17 pad 1: OUT -> Drain_Low
- TP20 pad 1: OUT -> Drain_Low
- TP23 pad 1: OUT -> Drain_Low
- TP3 pad 1: OUT -> GND2H
- TP7 pad 1: OUT -> GND2H
- U3 pad 1: Net-(C48-Pad1) -> Net-(U3-1Y)
- U3 pad 2: Net-(C54-Pad1) -> Net-(U3-1A)
- U3 pad 3: GND -> Net-(U3-1B)
- U3 pad 4: Net-(R47-Pad2) -> +3.3V
Routing:
- net OUT: track 68.8 -> 0.00 mm, vias 4 -> 17
- net IN+L: track 0.00 -> 64.8 mm, vias 0 -> 2
- net IN-L: track 0.00 -> 61.2 mm, vias 0 -> 2
- net HighERR: track 0.00 -> 54.7 mm, vias 0 -> 2
- net ~{RSTL}: track 2.33 -> 55.9 mm, vias 1 -> 2
- net IN+H: track 0.00 -> 53.5 mm, vias 0 -> 2
- net IN-H: track 0.00 -> 50.2 mm, vias 0 -> 2
- net ~{RSTH}: track 2.33 -> 51.8 mm, vias 1 -> 2
- net GND2H: track 0.00 -> 43.0 mm, vias 0 -> 35
- net Drain_Low: track 0.00 -> 38.4 mm, vias 0 -> 33
- net GND: track 17.0 -> 51.2 mm, vias 0 -> 15
- net ~{FLTL}: track 16.4 -> 48.2 mm, vias 1 -> 2
- net RDYL: track 17.5 -> 47.7 mm, vias 1 -> 2
- net ~{FLTH}: track 16.4 -> 44.1 mm, vias 1 -> 2
- net LowERR: track 0.00 -> 20.8 mm, vias 0 -> 1
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- added copper zone on In1.Cu, net +12V
- added copper zone on F.Cu, net +3.3V
- added copper zone on F.Cu, net Drain_Low
- added copper zone on In1.Cu, net Drain_Low
- added copper zone on B.Cu, net GND
- added copper zone on In2.Cu, net GND1
- added copper zone on B.Cu, net GND2H
- added copper zone on F.Cu, net GND2H
- added copper zone on In1.Cu, net GND2H
- added copper zone on F.Cu, net GNDPWR
- added copper zone on In1.Cu, net GNDPWR
- added copper zone on In2.Cu, net GNDPWR
- added copper zone on F.Cu, net OUT
- added copper zone on In1.Cu, net OUT
- added copper zone on In2.Cu, net OUT
- added copper zone on B.Cu, net VDC
- added copper zone on F.Cu, net VDC
- added copper zone on In1.Cu, net VDC
- added copper zone on In2.Cu, net VDC
Other:
- board outline added: 134.6 x 88.3 mm
