File: Тестовые драйвера.kicad_pcb (KiCad board)
At the start: 4 copper layers, 134.6 x 88.3 mm, 170 parts, among them J1 Conn_01x01, J2 Conn_01x01, J3 Conn_01x01, J4 Conn_01x01, J5 Conn_01x01, J6 Conn_02x10_Odd_Even, Q1 C2M0280120D, Q2 C2M0280120D, Q3 C2M0280120D, Q4 C2M0280120D, Q5 C2M0280120D, Q6 C2M0280120D, U3 HEF4082BT

Commit message: Пытаюсь сделать как у вольфспида
Parts:
- removed C13, C14: 0.1n, Capacitor_SMD:C_0805_2012Metric_Pad1.18x1.45mm_HandSolder
- removed C33: 1u, Capacitor_SMD:C_0805_2012Metric_Pad1.18x1.45mm_HandSolder
- removed C34: Cblk, Capacitor_SMD:C_0805_2012Metric_Pad1.18x1.45mm_HandSolder
- removed C47, C49, C50, C52, C53: 56p, Capacitor_SMD:C_0805_2012Metric_Pad1.18x1.45mm_HandSolder
- removed C55: 100n, Capacitor_SMD:C_0805_2012Metric_Pad1.18x1.45mm_HandSolder
- removed C56: Cf, Capacitor_SMD:C_0805_2012Metric_Pad1.18x1.45mm_HandSolder
- removed L3: 6.8u, Inductor_SMD:L_1812_4532Metric_Pad1.30x3.40mm_HandSolder
- removed PS1, PS2: A1215S-1WR3, Converter_DCDC:Converter_DCDC_XP_POWER-IAxxxxS_THT
- removed PS3: B1203S-1WR3, Converter_DCDC:Converter_DCDC_RECOM_R-78S-0.1_THT
- removed R10: 330, Resistor_SMD:R_0805_2012Metric_Pad1.20x1.40mm_HandSolder
- removed R22, R23, R55, R7: Rdesat, Resistor_SMD:R_0805_2012Metric_Pad1.20x1.40mm_HandSolder
- removed R24, R25, R8, R9: 4.7k, Resistor_SMD:R_0805_2012Metric_Pad1.20x1.40mm_HandSolder
- removed R52, R53, R54: 15, Resistor_SMD:R_1206_3216Metric_Pad1.30x1.75mm_HandSolder
- removed R56, R57: 0.5m, Shunt_My:LR2725
- removed R58: 1k, Resistor_SMD:R_0805_2012Metric_Pad1.20x1.40mm_HandSolder
- removed TP15, TP16, TP5, TP6: TestPoint, TestPoint:TestPoint_Loop_D2.50mm_Drill1.0mm_LowProfile
- removed U3: HEF4082BT, Package_SO:SO-14_3.9x8.65mm_P1.27mm
- added C44: Cf, Capacitor_SMD:C_0805_2012Metric_Pad1.18x1.45mm_HandSolder, F.Cu at (245.3, 35.1)
- added C45: 56p, Capacitor_SMD:C_0805_2012Metric_Pad1.18x1.45mm_HandSolder, F.Cu at (245.3, 38.1)
- added D17: ~, Mornsun:QAxCx, F.Cu at (246.3, 113.6)
- added Q7: ~, Package_TO_SOT_SMD:SOT-23, F.Cu at (79.4, 166.9)
- C1, C15, C20, C6: value 0.47u -> 10u; footprint Capacitor_SMD:C_1210_3225Metric_Pad1.33x2.70mm_HandSolder -> Capacitor_SMD:C_1206_3216Metric_Pad1.33x1.80mm_HandSolder; moved to F.Cu
- C10: value 100n -> Cf; moved to F.Cu
- C11: value Cf -> 100p; footprint Capacitor_SMD:C_0805_2012Metric_Pad1.18x1.45mm_HandSolder -> Capacitor_SMD:C_1206_3216Metric_Pad1.33x1.80mm_HandSolder; moved to F.Cu
- C12: value Cblk -> 100p
- C16, C17, C2, C3: footprint Capacitor_SMD:C_0805_2012Metric_Pad1.18x1.45mm_HandSolder -> Capacitor_SMD:C_1206_3216Metric_Pad1.33x1.80mm_HandSolder
- C18, C19, C4, C5: footprint Capacitor_SMD:C_1210_3225Metric_Pad1.33x2.70mm_HandSolder -> Capacitor_SMD:C_1206_3216Metric_Pad1.33x1.80mm_HandSolder; moved to F.Cu
- C21, C41: value 100n -> 10n; moved to F.Cu
- C22, C42, R21: moved to F.Cu
- C23: value CY-270p -> 100p; footprint Capacitor_SMD:C_1210_3225Metric_Pad1.33x2.70mm_HandSolder -> Capacitor_SMD:C_1206_3216Metric_Pad1.33x1.80mm_HandSolder
- C24: value 4.7u -> 10u; footprint Capacitor_SMD:C_1210_3225Metric_Pad1.33x2.70mm_HandSolder -> Capacitor_SMD:C_1206_3216Metric_Pad1.33x1.80mm_HandSolder
- C25: value 4.7u -> 0.1u; footprint Capacitor_SMD:C_1210_3225Metric_Pad1.33x2.70mm_HandSolder -> Capacitor_SMD:C_1206_3216Metric_Pad1.33x1.80mm_HandSolder
- C26: value 10u -> 10n; footprint Capacitor_SMD:C_1210_3225Metric_Pad1.33x2.70mm_HandSolder -> Capacitor_SMD:C_0805_2012Metric_Pad1.18x1.45mm_HandSolder; moved to F.Cu
- C27: value 10u -> Cf; moved to F.Cu
- C28: value 0.1u -> 10u; footprint Capacitor_SMD:C_0805_2012Metric_Pad1.18x1.45mm_HandSolder -> Capacitor_SMD:C_1210_3225Metric_Pad1.33x2.70mm_HandSolder; moved to F.Cu
- C29: value 100n -> 10u; footprint Capacitor_SMD:C_0805_2012Metric_Pad1.18x1.45mm_HandSolder -> Capacitor_SMD:C_1210_3225Metric_Pad1.33x2.70mm_HandSolder; moved to F.Cu
- C30: value Cf -> 0.1u; moved to F.Cu
- C31: value CY-270p -> 1u; footprint Capacitor_SMD:C_1210_3225Metric_Pad1.33x2.70mm_HandSolder -> Capacitor_SMD:C_0805_2012Metric_Pad1.18x1.45mm_HandSolder; moved to F.Cu
- C32: value 0.1u -> 100p
- C35: value 0.1n -> 10u; footprint Capacitor_SMD:C_0805_2012Metric_Pad1.18x1.45mm_HandSolder -> Capacitor_SMD:C_1206_3216Metric_Pad1.33x1.80mm_HandSolder; moved to F.Cu
- C36: value 0.1n -> 0.1u; footprint Capacitor_SMD:C_0805_2012Metric_Pad1.18x1.45mm_HandSolder -> Capacitor_SMD:C_1206_3216Metric_Pad1.33x1.80mm_HandSolder; moved to F.Cu
- C37: value 10u -> 10n; moved to F.Cu
- C38: value 0.1u -> Cf; moved to F.Cu
- C39: value 100n -> 2.2u; moved to F.Cu
- C40: value Cf -> 2.2u; moved to F.Cu
- C43: value 1u -> 10n; moved to F.Cu
- C9: value CY-270p -> 10n; footprint Capacitor_SMD:C_1210_3225Metric_Pad1.33x2.70mm_HandSolder -> Capacitor_SMD:C_0805_2012Metric_Pad1.18x1.45mm_HandSolder
- D10, D2: footprint Diode_SMD:D_SMA_Handsoldering -> Diode_SMD:D_SMB_Handsoldering; moved to B.Cu
- D11: value D_Zener_Small -> D_Small; footprint Diode_SMD:D_SMA-SMB_Universal_Handsoldering -> Diode_SMD:D_SMB_Handsoldering
- D12: value D_Zener_Small -> ~; footprint Diode_SMD:D_SMA-SMB_Universal_Handsoldering -> Package_SO:SOIC-8_3.9x4.9mm_P1.27mm
- D13: value LED_Small -> ~; footprint LED_SMD:LED_0805_2012Metric_Pad1.15x1.40mm_HandSolder -> Package_TO_SOT_SMD:SOT-23-5
- D14: value LED_Small -> ~
- D15: value MBR0520 -> ~; footprint Diode_My:D_SOD_123_Hand -> LED_SMD:LED_0805_2012Metric_Pad1.15x1.40mm_HandSolder
- D16: value MBR0520 -> ~; footprint Diode_My:D_SOD_123_Hand -> Mornsun:QAxCx
- D3, D9: value D_Small -> D_Zener_Small; footprint Diode_SMD:D_SMA_Handsoldering -> Diode_SMD:D_SOD-323_HandSoldering
- D4, D5: value D_Zener_Small -> ~; footprint Diode_SMD:D_SMA-SMB_Universal_Handsoldering -> Diode_SMD:D_SOD-123
- D6: value LED_Small -> ~; footprint LED_SMD:LED_0805_2012Metric_Pad1.15x1.40mm_HandSolder -> Mornsun:K78xxM-1000R3
- D7: value LED_Small -> NSI6651; footprint LED_SMD:LED_0805_2012Metric_Pad1.15x1.40mm_HandSolder -> Package_SO:SOIC-16W_7.5x10.3mm_P1.27mm
- D8: value NSI6651 -> D_Small; footprint Package_SO:SOIC-16W_7.5x10.3mm_P1.27mm -> Diode_SMD:D_SMA_Handsoldering
- J6: value Conn_02x10_Odd_Even -> ~; footprint Connector_PinSocket_2.54mm:PinSocket_2x10_P2.54mm_Vertical -> Connector_Molex:Molex_Micro-Fit_3.0_43045-1212_2x06_P3.00mm_Vertical
- L1, L2: value 6.8u -> 22u; moved to F.Cu
- Q1, Q2, Q3, Q4, Q5, Q6: footprint Package_TO_SOT_THT:TO-220-3_Horizontal_TabUp -> Package_TO_SOT_THT:TO-247-3_Horizontal_TabUp
- R11, R26: value 330 -> 15; footprint Resistor_SMD:R_0805_2012Metric_Pad1.20x1.40mm_HandSolder -> Resistor_SMD:R_1206_3216Metric_Pad1.30x1.75mm_HandSolder
- R14, R19, R33, R38, R4: value 15 -> Rdesat; footprint Resistor_SMD:R_1206_3216Metric_Pad1.30x1.75mm_HandSolder -> Resistor_SMD:R_0805_2012Metric_Pad1.20x1.40mm_HandSolder
- R16, R36, R5: value Rdesat -> 15; footprint Resistor_SMD:R_0805_2012Metric_Pad1.20x1.40mm_HandSolder -> Resistor_SMD:R_1206_3216Metric_Pad1.30x1.75mm_HandSolder; moved to F.Cu
- R27: value 330 -> 0
- R31: value 0 -> 15; footprint Resistor_SMD:R_0805_2012Metric_Pad1.20x1.40mm_HandSolder -> Resistor_SMD:R_1206_3216Metric_Pad1.30x1.75mm_HandSolder
- R40: value 15 -> 120; footprint Resistor_SMD:R_1206_3216Metric_Pad1.30x1.75mm_HandSolder -> Resistor_SMD:R_0805_2012Metric_Pad1.20x1.40mm_HandSolder
- R41: value Rdesat -> 1k; moved to F.Cu
- R42: value 120 -> 4.7k
- R43, R44, R45: value 120 -> 15; footprint Resistor_SMD:R_0805_2012Metric_Pad1.20x1.40mm_HandSolder -> Resistor_SMD:R_1206_3216Metric_Pad1.30x1.75mm_HandSolder
- R46: value 120 -> Rdesat
- R47: value 2k -> 15; footprint Resistor_SMD:R_0805_2012Metric_Pad1.20x1.40mm_HandSolder -> Resistor_SMD:R_1206_3216Metric_Pad1.30x1.75mm_HandSolder
- R48, R50: value 120 -> 1k
- R49: value 120 -> 10k
- R51: value 15 -> 560; footprint Resistor_SMD:R_1206_3216Metric_Pad1.30x1.75mm_HandSolder -> Resistor_SMD:R_0805_2012Metric_Pad1.20x1.40mm_HandSolder
- moved TP23 216.2 mm to (250.0, 46.7)
- moved TP24 209.0 mm to (250.0, 51.3)
- moved D9 206.6 mm to (258.4, 157.9), turned to 0 degrees
- moved TP22 206.3 mm to (250.0, 42.0)
- moved TP25 205.1 mm to (250.0, 56.0)
- moved TP1 204.5 mm to (245.8, 151.9)
- moved D11 203.7 mm to (271.1, 123.5), turned to 0 degrees
- moved TP8 202.5 mm to (245.8, 156.6)
- moved TP11 200.7 mm to (245.8, 161.2)
- moved TP17 199.0 mm to (245.8, 165.8)
- moved TP20 197.6 mm to (245.8, 170.5)
- moved TP12 196.0 mm to (245.3, 42.0)
- moved TP21 195.5 mm to (245.3, 65.3)
- moved TP18 195.0 mm to (245.3, 56.0)
- moved D5 193.6 mm to (270.4, 95.0), turned to 0 degrees
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Connections:
- C10 pad 1: ClampH -> Net-(C10-Pad1)
- C11 pad 1: Net-(C11-Pad1) -> Net-(D16-Vin)
- C11 pad 2: GND2H -> GND1
- C16 pad 1: -15VH -> -4VH
- C17 pad 1: -15VH -> -4VH
- C18 pad 1: +12V -> +15V
- C19 pad 1: Net-(PS2-+Vin) -> Net-(D17-Vin)
- C23 pad 1: GND1 -> Net-(D17-Vin)
- C23 pad 2: GNDPWR -> GND1
- C24 pad 1: +12V -> GNDPWR
- C24 pad 2: GND1 -> +15VL
- C25 pad 1: Net-(PS3-+Vin) -> GNDPWR
- C25 pad 2: GND1 -> +15VL
- C26 pad 1: +3.3V -> ClampH
- C26 pad 2: GND -> GND2H
- C27 pad 1: GNDPWR -> Net-(C27-Pad1)
- C27 pad 2: +15VL -> GND2H
- C28 pad 1: GNDPWR -> +15V
- C28 pad 2: +15VL -> GND
- C29 pad 1: ClampH -> +5V
- C29 pad 2: GND2H -> GND
- C30 pad 1: Net-(C30-Pad1) -> GND
- C30 pad 2: GND2H -> +5V
- C31 pad 1: GND1 -> GND
- C31 pad 2: GND -> +5V
- C32 pad 1: GND -> GNDPWR
- C32 pad 2: +3.3V -> Net-(D5-K)
- C35 pad 1: ~{FLTL} -> -15VL
- C35 pad 2: GND -> GNDPWR
- C36 pad 1: RDYL -> -15VL
- C36 pad 2: GND -> GNDPWR
- C37 pad 1: -15VL -> ClampL
- C38 pad 1: -15VL -> Net-(C38-Pad1)
- C39 pad 1: ClampL -> +5V
- C39 pad 2: GNDPWR -> GND
- C4 pad 1: +12V -> +15V
- C40 pad 1: Net-(C40-Pad1) -> +5V
- C40 pad 2: GNDPWR -> GND
- C43 pad 1: +3.3V -> ClampL
- C43 pad 2: GND -> GNDPWR
- C46 pad 1: Net-(U3-1A) -> ~{FLT}
- C5 pad 1: Net-(PS1-+Vin) -> Net-(D16-Vin)
- C6 pad 2: -15VH -> -4VH
- C7 pad 2: +3.3V -> +5V
- C8 pad 2: +3.3V -> +5V
- C9 pad 1: GND1 -> ClampH
- D1 pad 1: -15VH -> -4VH
- D1 pad 10: IN+H -> PWM_P
- D1 pad 11: IN-H -> PWM_N
- D1 pad 12: RDYH -> RDY
- D1 pad 13: ~{FLTH} -> ~{FLT}
- D1 pad 14: ~{RSTH} -> RST
- D1 pad 15: +3.3V -> +5V
- D1 pad 8: -15VH -> -4VH
- D10 pad 1: Net-(D10-K) -> VDC
- D11 pad 1: Net-(D11-K) -> Drain_Low
- D11 pad 2: Net-(D10-A) -> Net-(D11-A)
- D12 pad 1: Net-(D12-K) -> unconnected-(D12-RO-Pad1)
- D12 pad 2: Net-(D11-K) -> +5V
- D13 pad 1: GND -> RDY
- D13 pad 2: Net-(D13-A) -> ~{FLT}
- D14 pad 1: Net-(D14-K) -> ~{FLT}
- D14 pad 2: +3.3V -> Net-(D14-A)
- D15 pad 1: Net-(D15-K) -> GND
- D15 pad 2: HighERR -> Net-(D15-A)
- D16 pad 1: Net-(D16-K) -> Net-(D16-Vin)
- D16 pad 2: LowERR -> GND1
- D2 pad 1: VDC -> Net-(D10-A)
- D3 pad 1: Net-(D2-A) -> Net-(D3-K)
- D3 pad 2: Net-(D3-A) -> Net-(D2-A)
- D4 pad 1: Net-(D4-K) -> Net-(D1-DESAT)
- D4 pad 2: Net-(D3-A) -> GND2H
- D5 pad 2: Net-(D4-K) -> GNDPWR
- D6 pad 1: GND -> +15V
- D6 pad 2: Net-(D6-A) -> GND
- D7 pad 1: Net-(D7-K) -> -15VL
- D7 pad 2: +3.3V -> Net-(D5-K)
- D8 pad 1: -15VL -> Net-(D11-A)
- D8 pad 2: Net-(D8-DESAT) -> Net-(D8-A)
- D9 pad 1: Drain_Low -> Net-(D9-K)
- D9 pad 2: Net-(D10-K) -> Net-(D8-A)
- J6 pad 1: +3.3V -> unconnected-(J6-Pin_1-Pad1)
- J6 pad 10: HighERR -> Fault_N
- J6 pad 11: GND -> unconnected-(J6-Pin_11-Pad11)
- J6 pad 12: LowERR_ADC -> unconnected-(J6-Pin_12-Pad12)
- J6 pad 2: ~{RSTH} -> +15V
- J6 pad 3: +3.3V -> PWM_P
- J6 pad 4: IN+H -> Fault_P
- J6 pad 5: +3.3V -> unconnected-(J6-Pin_5-Pad5)
- J6 pad 6: IN-H -> Reset
- J6 pad 7: +3.3V -> unconnected-(J6-Pin_7-Pad7)
- J6 pad 8: LowERR -> GND
- J6 pad 9: +3.3V -> PWM_N
- L1 pad 1: +12V -> +15V
- L1 pad 2: Net-(PS1-+Vin) -> Net-(D16-Vin)
- L2 pad 1: +12V -> +15V
- L2 pad 2: Net-(PS2-+Vin) -> Net-(D17-Vin)
- R1 pad 2: Net-(R1-Pad2) -> ClampH
- R11 pad 1: ~{FLTH} -> OutH1
- R11 pad 2: Net-(D7-K) -> ClampH
- R12 pad 2: Net-(R12-Pad2) -> ClampH
- R13 pad 1: Net-(R12-Pad2) -> ClampH
- R13 pad 2: ClampH -> OutL1
- R14 pad 1: Net-(R14-Pad1) -> Net-(C22-Pad1)
- R14 pad 2: OutL1 -> ClampH
- R15 pad 2: Net-(R14-Pad1) -> OutL1
- R16 pad 1: Net-(C22-Pad1) -> OutH1
- R17 pad 2: Net-(R17-Pad2) -> ClampH
- R18 pad 1: Net-(R17-Pad2) -> ClampH
- R18 pad 2: ClampH -> OutL1
- R19 pad 1: Net-(R19-Pad1) -> Net-(C27-Pad1)
- R19 pad 2: OutL1 -> ClampH
- R2 pad 1: Net-(R1-Pad2) -> OutH1
- R20 pad 2: Net-(R19-Pad1) -> OutL1
- R21 pad 1: Net-(C30-Pad1) -> Net-(D9-K)
- R21 pad 2: ClampH -> Net-(D5-K)
- R26 pad 1: RDYL -> OutH2
- R26 pad 2: Net-(D13-A) -> ClampL
- R27 pad 1: ~{FLTL} -> IN+H
- R27 pad 2: Net-(D14-K) -> IN-L
- R28 pad 1: IN+H -> IN-H
- R28 pad 2: IN-L -> IN+L
- R29 pad 1: IN-H -> ~{RSTL}
- R3 pad 1: Net-(R3-Pad1) -> ClampH
- R30 pad 1: ~{RSTL} -> ~{RSTH}
- R30 pad 2: IN+L -> IN+H
- R31 pad 1: ~{RSTH} -> OutH2
- R31 pad 2: IN+H -> ClampL
- R32 pad 1: OutH2 -> ClampL
- R32 pad 2: Net-(R32-Pad2) -> OutL2
- R33 pad 1: Net-(R32-Pad2) -> Net-(C38-Pad1)
- R34 pad 1: Net-(R34-Pad1) -> ClampL
- R35 pad 1: ClampL -> OutH2
- R35 pad 2: Net-(R34-Pad1) -> ClampL
- R36 pad 1: Net-(C40-Pad1) -> OutH2
- R37 pad 1: OutH2 -> ClampL
- R37 pad 2: Net-(R37-Pad2) -> OutL2
- R38 pad 1: Net-(R37-Pad2) -> Net-(C42-Pad1)
- R39 pad 1: Net-(R39-Pad1) -> ClampL
- R4 pad 1: ClampH -> Net-(C10-Pad1)
- R4 pad 2: Net-(R3-Pad1) -> ClampH
- R40 pad 1: ClampL -> Fault_N
- R40 pad 2: Net-(R39-Pad1) -> Fault_P
- R41 pad 1: Net-(C42-Pad1) -> RST
- R41 pad 2: ClampL -> +5V
- R42 pad 1: Net-(U3-1A) -> Reset
- R42 pad 2: RDYH -> Net-(Q7-G)
- R43 pad 1: Net-(U3-2A) -> OutH2
- R43 pad 2: RDYL -> ClampL
- R44 pad 1: Net-(D15-K) -> OutH2
- R44 pad 2: HighERR_ADC -> ClampL
- R45 pad 1: HighERR -> ClampL
- R45 pad 2: Net-(U3-1Y) -> OutL2
- R46 pad 1: LowERR -> Net-(C44-Pad1)
- R46 pad 2: Net-(U3-2Y) -> ClampL
- R47 pad 1: GND -> ClampL
- R47 pad 2: HighERR_ADC -> OutL2
- R48 pad 1: Net-(U3-1B) -> RDY
- R48 pad 2: ~{FLTH} -> +5V
- R49 pad 1: Net-(U3-2B) -> ~{FLT}
- R49 pad 2: ~{FLTL} -> +5V
- R5 pad 1: Net-(C11-Pad1) -> ClampH
- R5 pad 2: ClampH -> OutL1
- R50 pad 1: Net-(D16-K) -> Net-(D14-A)
- R50 pad 2: LowERR_ADC -> +5V
- R51 pad 1: OutH2 -> Net-(D15-A)
- R51 pad 2: Net-(R51-Pad2) -> RDY
- R6 pad 1: Net-(D5-K) -> Net-(D3-K)
- R6 pad 2: Net-(R6-Pad2) -> Net-(D1-DESAT)
- TP14 pad 1: Net-(D8-DESAT) -> Net-(D5-K)
- TP17 pad 1: Drain_Low -> GNDPWR
- TP18 pad 1: ClampL -> Drain_Low
- TP19 pad 1: GNDPWR -> ClampL
- TP20 pad 1: Drain_Low -> GNDPWR
- TP21 pad 1: ClampL -> Drain_Low
- TP22 pad 1: GNDPWR -> ClampL
- TP23 pad 1: Drain_Low -> GNDPWR
- TP24 pad 1: ClampL -> Drain_Low
- TP25 pad 1: GNDPWR -> ClampL
- TP7 pad 1: GND2H -> VDC
- TP8 pad 1: VDC -> GND2H
Routing:
- net ClampL: track 123.8 -> 0.34 mm, vias 1 -> 0
- net IN+L: track 64.8 -> 0.00 mm, vias 2 -> 0
- net IN-L: track 61.2 -> 0.00 mm, vias 2 -> 0
- net ~{RSTL}: track 55.9 -> 0.00 mm, vias 2 -> 0
- net HighERR: track 54.7 -> 0.00 mm, vias 2 -> 0
- net IN+H: track 53.5 -> 0.00 mm, vias 2 -> 0
- net ~{RSTH}: track 51.8 -> 0.00 mm, vias 2 -> 0
- net GND: track 51.2 -> 0.00 mm, vias 15 -> 0
- net IN-H: track 50.2 -> 0.00 mm, vias 2 -> 0
- net GND1: track 49.9 -> 0.00 mm, vias 3 -> 0
- net ~{FLTL}: track 48.2 -> 0.00 mm, vias 2 -> 0
- net GNDPWR: track 48.2 -> 0.00 mm, vias 56 -> 0
- net RDYL: track 47.7 -> 0.00 mm, vias 2 -> 0
- net ~{FLTH}: track 44.1 -> 0.00 mm, vias 2 -> 0
- net GND2H: track 43.0 -> 0.00 mm, vias 35 -> 7
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- added copper zone on F.Cu, net +15VH
- added copper zone on B.Cu, net -4VH
- added copper zone on F.Cu, net -4VH
- added copper zone on In2.Cu, net -4VH
- added copper zone on F.Cu, net ClampH
- added copper zone on In2.Cu, net OutL1
- removed copper zone on In1.Cu, net +12V
- removed copper zone on B.Cu, net +15VL
- removed copper zone on F.Cu, net +3.3V
- removed copper zone on In2.Cu, net -15VH
- removed copper zone on In2.Cu, net -15VL
- removed copper zone on F.Cu, net Drain_Low
- removed copper zone on In1.Cu, net Drain_Low
- removed copper zone on B.Cu, net GND
- removed copper zone on In2.Cu, net GND1
- removed copper zone on B.Cu, net GNDPWR
- removed copper zone on F.Cu, net GNDPWR
- removed copper zone on In1.Cu, net GNDPWR
- removed copper zone on In2.Cu, net GNDPWR
- removed copper zone on F.Cu, net Net-(R1-Pad2)
- removed copper zone on B.Cu, net Net-(R12-Pad2)
- removed copper zone on F.Cu, net Net-(R14-Pad1)
- removed copper zone on B.Cu, net Net-(R17-Pad2)
- removed copper zone on F.Cu, net Net-(R19-Pad1)
- removed copper zone on F.Cu, net Net-(R3-Pad1)
- removed copper zone on F.Cu, net Net-(R32-Pad2)
- removed copper zone on F.Cu, net Net-(R34-Pad1)
- removed copper zone on B.Cu, net Net-(R37-Pad2)
- removed copper zone on F.Cu, net Net-(R39-Pad1)
- removed copper zone on B.Cu, net Net-(R51-Pad2)
- removed copper zone on F.Cu, net Net-(R53-Pad1)
- removed copper zone on B.Cu, net OUT
- removed copper zone on F.Cu, net OUT
- removed copper zone on In1.Cu, net OUT
- removed copper zone on In2.Cu, net OUT
- removed copper zone on F.Cu, net OutH2
- removed copper zone on F.Cu, net OutL2
- removed copper zone on B.Cu, net VDC
- removed copper zone on F.Cu, net VDC
- removed copper zone on In1.Cu, net VDC
- removed copper zone on In2.Cu, net VDC
Other:
- board size 134.6 x 88.3 mm -> 134.6 x 105.3 mm

Commit message: VER1.0: пробую уложиться в ширину транзисторов
Parts:
- removed C10, C22, C27, C38, C42, C44: Cf, Capacitor_SMD:C_0805_2012Metric_Pad1.18x1.45mm_HandSolder
- removed TP1, TP10, TP11, TP12, TP13, TP14, TP17, TP18, TP19, TP2, TP20, TP21, TP22, TP23, TP24, TP25, TP26, TP3, TP4, TP7, TP8, TP9: TestPoint, TestPoint:TestPoint_Loop_D2.50mm_Drill1.0mm_LowProfile
- C16, C17, C2, C3, D10, D2: moved to F.Cu
- moved J6 115.9 mm to (101.0, 113.3)
- moved L1 50.6 mm to (140.0, 106.8), turned to 90 degrees
- moved D16 47.8 mm to (130.8, 114.6), turned to 0 degrees
- moved C4 46.6 mm to (144.8, 108.8), turned to 0 degrees
- moved C5 43.6 mm to (144.8, 106.0), turned to 0 degrees
- moved Q4 42.2 mm to (101.9, 70.0)
- moved Q5 42.2 mm to (101.9, 87.0)
- moved Q6 42.2 mm to (101.9, 104.0)
- moved C11 40.1 mm to (144.8, 103.2), turned to 0 degrees
- moved D2 35.8 mm to (128.2, 53.2)
- moved D10 31.3 mm to (117.5, 53.2)
- moved C6 24.6 mm to (138.8, 89.5), turned to -90 degrees
- moved C21 22.3 mm to (120.4, 88.0), turned to 180 degrees
- moved C26 22.3 mm to (120.4, 105.0), turned to 180 degrees
- moved C9 22.3 mm to (120.4, 71.0), turned to 180 degrees
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Connections:
- R14 pad 1: Net-(C22-Pad1) -> GND2H
- R19 pad 1: Net-(C27-Pad1) -> GND2H
- R33 pad 1: Net-(C38-Pad1) -> GNDPWR
- R38 pad 1: Net-(C42-Pad1) -> GNDPWR
- R4 pad 1: Net-(C10-Pad1) -> GND2H
- R46 pad 1: Net-(C44-Pad1) -> GNDPWR
Routing:
- net VDC: track 8.24 -> 18.5 mm
- net -4VH: track 0.00 -> 4.96 mm, vias 8 -> 1
- net ClampH: track 86.6 -> 91.0 mm
- net Net-(D2-A): track 15.6 -> 11.4 mm, vias 1 -> 0
- net +15VH: track 0.00 -> 3.44 mm, vias 4 -> 1
- net GND2H: track 0.00 -> 3.40 mm, vias 7 -> 1
- net OutL1: track 0.00 -> 1.98 mm
- net Net-(D10-A): track 6.55 -> 5.75 mm
- removed copper zone on B.Cu, net +15VH
- removed copper zone on B.Cu, net -4VH
- removed copper zone on In2.Cu, net -4VH
- removed copper zone on B.Cu, net GND2H
Other:
- board size 134.6 x 105.3 mm -> 95.7 x 77.6 mm

Commit message: Пытаюсь уложиться в контур транзисторов
Parts:
- removed C1, C15, C20, C6: 10u, Capacitor_SMD:C_1206_3216Metric_Pad1.33x1.80mm_HandSolder
- C11, C16, C17, C4, C5, L1: moved to B.Cu
- J1, J2, J3: footprint Connector_Power_My:Cuprum_M4 -> Bush_my:Bush_SMD_M3
- moved D17 158.8 mm to (87.5, 113.9), turned to 180 degrees
- moved J1 61.9 mm to (106.0, 98.5)
- moved J3 60.5 mm to (106.0, 65.0)
- moved J2 59.7 mm to (106.0, 81.5)
- moved C8 55.8 mm to (119.5, 115.5), turned to 90 degrees
- moved C7 53.0 mm to (122.0, 115.5), turned to 90 degrees
- moved C16 46.6 mm to (139.5, 116.0), turned to 90 degrees
- moved C17 46.6 mm to (137.0, 116.0), turned to 90 degrees
- moved D1 39.1 mm to (129.5, 112.0), turned to 180 degrees
- moved C3 38.8 mm to (139.5, 113.0), turned to 90 degrees
- moved C2 38.2 mm to (137.0, 113.0), turned to 90 degrees
- moved C11 32.7 mm to (119.5, 124.0), turned to -90 degrees
- moved C5 28.6 mm to (122.5, 124.0), turned to -90 degrees
- moved C4 24.6 mm to (125.5, 124.0), turned to -90 degrees
- moved L1 20.5 mm to (129.0, 124.0), turned to -90 degrees
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Connections:
- C12 pad 1: GND2H -> OUT
- C16 pad 2: GND2H -> OUT
- C17 pad 2: GND2H -> OUT
- C2 pad 1: GND2H -> OUT
- C21 pad 2: GND2H -> OUT
- C26 pad 2: GND2H -> OUT
- C3 pad 1: GND2H -> OUT
- C9 pad 2: GND2H -> OUT
- D1 pad 3: GND2H -> OUT
- D16 pad 6: GND2H -> OUT
- D4 pad 2: GND2H -> OUT
- Q1 pad 3: GND2H -> OUT
- Q2 pad 3: GND2H -> OUT
- Q3 pad 3: GND2H -> OUT
- Q4 pad 2: Drain_Low -> OUT
- Q5 pad 2: Drain_Low -> OUT
- Q6 pad 2: Drain_Low -> OUT
- R14 pad 1: GND2H -> OUT
- R19 pad 1: GND2H -> OUT
- R4 pad 1: GND2H -> OUT
Routing:
- net Net-(D1-DESAT): track 10.7 -> 69.0 mm, vias 0 -> 1
- net VDC: track 18.5 -> 0.00 mm
- net OUT: track 0.00 -> 14.0 mm
- net +15VH: track 3.44 -> 17.2 mm, vias 1 -> 0
- net -4VH: track 4.96 -> 18.5 mm, vias 1 -> 0
- net Net-(D2-A): track 11.4 -> 0.00 mm
- net ClampH: track 91.0 -> 84.6 mm, vias 1 -> 2
- net Net-(D10-A): track 5.75 -> 0.00 mm
- net GND2H: track 3.40 -> 0.00 mm, vias 1 -> 0
- net Net-(D3-K): track 2.75 -> 0.00 mm
- net OutL1: track 1.98 -> 1.19 mm
- added copper zone on B.Cu, net OutL1
- removed copper zone on F.Cu, net +15VH
- removed copper zone on F.Cu, net -4VH
- removed copper zone on F.Cu, net ClampH
- removed copper zone on F.Cu, net GND2H
- removed copper zone on In1.Cu, net GND2H
- removed copper zone on F.Cu, net OutL1
- removed copper zone on In2.Cu, net OutL1
Other:
- board size 95.7 x 77.6 mm -> 72.7 x 84.6 mm
