File: Тестовые драйвера.kicad_pcb (KiCad board)
At the start: 2 copper layers, 114.4 x 54.6 mm, 117 parts, among them J1 Conn_01x01, J10 Conn_01x01, J11 Conn_01x01, J12 Conn_01x01, J13 Conn_01x01, J14 Conn_01x03, J15 Conn_01x03, J16 Conn_01x03, J2 Conn_01x01, J3 Conn_01x01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

Commit message: VER1.0.2: развел нижнюю сторону
Parts:
- removed C11, C23: 100p, Capacitor_SMD:C_1206_3216Metric_Pad1.33x1.80mm_HandSolder
- removed C12, C32: 100p, Capacitor_SMD:C_0805_2012Metric_Pad1.18x1.45mm_HandSolder
- removed C16, C2, C24, C35: 10u, Capacitor_SMD:C_1206_3216Metric_Pad1.33x1.80mm_HandSolder
- removed C17, C25, C3, C36: 0.1u, Capacitor_SMD:C_1206_3216Metric_Pad1.33x1.80mm_HandSolder
- removed C18, C19, C4, C5: 4.7u, Capacitor_SMD:C_1206_3216Metric_Pad1.33x1.80mm_HandSolder
- removed C28, C29: 10u, Capacitor_SMD:C_1210_3225Metric_Pad1.33x2.70mm_HandSolder
- removed C30, C7: 0.1u, Capacitor_SMD:C_0805_2012Metric_Pad1.18x1.45mm_HandSolder
- removed C31, C8: 1u, Capacitor_SMD:C_0805_2012Metric_Pad1.18x1.45mm_HandSolder
- removed C39, C40: 2.2u, Capacitor_SMD:C_0805_2012Metric_Pad1.18x1.45mm_HandSolder
- removed C45, C46: 56p, Capacitor_SMD:C_0805_2012Metric_Pad1.18x1.45mm_HandSolder
- removed D1, D7: NSI6651, Package_SO:SOIC-16W_7.5x10.3mm_P1.27mm
- removed D10, D11, D2: D_Small, Diode_SMD:D_SMB_Handsoldering
- removed D12: ~, Package_SO:SOIC-8_3.9x4.9mm_P1.27mm
- removed D13: ~, Package_TO_SOT_SMD:SOT-23-5
- removed D14, D15: ~, LED_SMD:LED_0805_2012Metric_Pad1.15x1.40mm_HandSolder
- removed D16, D17: ~, Mornsun:QAxCx
- removed D3, D9: D_Zener_Small, Diode_SMD:D_SOD-323_HandSoldering
- removed D4, D5: ~, Diode_SMD:D_SOD-123
- removed D6: ~, Mornsun:K78xxM-1000R3
- removed D8: D_Small, Diode_SMD:D_SMA_Handsoldering
- removed J12, J13, J8, J9: Conn_01x01, Bush_my:Bush_5x3
- removed J14, J15, J16: Conn_01x03, Bush_my:247_border_my
- removed J6: ~, Connector_Molex:Molex_Micro-Fit_3.0_43045-1212_2x06_P3.00mm_Vertical
- removed L1, L2: 22u, Inductor_SMD:L_1812_4532Metric_Pad1.30x3.40mm_HandSolder
- removed Q7: ~, Package_TO_SOT_SMD:SOT-23
- removed R21, R6: Rdesat, Resistor_SMD:R_0805_2012Metric_Pad1.20x1.40mm_HandSolder
- removed R27, R28, R29, R30: 0, Resistor_SMD:R_0805_2012Metric_Pad1.20x1.40mm_HandSolder
- removed R40: 120, Resistor_SMD:R_0805_2012Metric_Pad1.20x1.40mm_HandSolder
- removed R41, R48, R50: 1k, Resistor_SMD:R_0805_2012Metric_Pad1.20x1.40mm_HandSolder
- removed R42: 4.7k, Resistor_SMD:R_0805_2012Metric_Pad1.20x1.40mm_HandSolder
- removed R49: 10k, Resistor_SMD:R_0805_2012Metric_Pad1.20x1.40mm_HandSolder
- removed R51: 560, Resistor_SMD:R_0805_2012Metric_Pad1.20x1.40mm_HandSolder
- J4: footprint Connector_PinSocket_2.54mm:PinSocket_1x04_P2.54mm_Vertical -> Connector_PinSocket_2.54mm:PinSocket_2x04_P2.54mm_Vertical
- J5: value Conn_01x04 -> Conn_02x05_Odd_Even; footprint Connector_PinSocket_2.54mm:PinSocket_1x04_P2.54mm_Vertical -> Connector_PinSocket_2.54mm:PinSocket_2x05_P2.54mm_Vertical
- J7: value Conn_01x04 -> Conn_01x01; footprint Connector_PinSocket_2.54mm:PinSocket_1x04_P2.54mm_Vertical -> Bush_my:Bush_5x3; moved to F.Cu
- moved J7 73.6 mm to (349.5, 289.8), turned to 90 degrees
- moved J3 36.1 mm to (349.5, 306.8), turned to 90 degrees
- moved J4 31.6 mm to (370.0, 316.8), turned to 90 degrees
- moved J5 31.1 mm to (320.2, 317.0), turned to 90 degrees
- moved J1 12.6 mm to (349.5, 272.8), turned to 90 degrees
- moved C21 5.00 mm to (361.4, 296.3)
- moved C26 5.00 mm to (361.4, 313.3)
- moved C9 5.00 mm to (361.4, 279.3)
- moved Q1 5.00 mm to (356.4, 267.2)
- moved Q2 5.00 mm to (356.4, 284.2)
- moved Q3 5.00 mm to (356.4, 301.2)
- moved R1 5.00 mm to (364.1, 274.8)
- moved R11 5.00 mm to (364.0, 291.8)
- moved R12 5.00 mm to (364.0, 289.3)
- moved R13 5.00 mm to (364.0, 286.8)
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Connections:
- C37 pad 2: Drain_Low -> GNDPWR
- C41 pad 2: Drain_Low -> GNDPWR
- C43 pad 2: Drain_Low -> GNDPWR
- J1 pad 1: Drain_Low -> OUT
- J3 pad 1: VDC -> OUT
- J5 pad 1: unconnected-(J5-Pin_1-Pad1) -> GNDPWR
- J5 pad 2: unconnected-(J5-Pin_2-Pad2) -> GNDPWR
- J5 pad 3: unconnected-(J5-Pin_3-Pad3) -> OutH2
- J5 pad 4: unconnected-(J5-Pin_4-Pad4) -> OutH2
- J7 pad 1: unconnected-(J7-Pin_1-Pad1) -> OUT
- Q4 pad 3: Drain_Low -> GNDPWR
- Q5 pad 3: Drain_Low -> GNDPWR
- Q6 pad 3: Drain_Low -> GNDPWR
- R33 pad 1: Drain_Low -> GNDPWR
- R38 pad 1: Drain_Low -> GNDPWR
- R46 pad 1: Drain_Low -> GNDPWR
Routing:
- net OUT: track 0.00 -> 26.0 mm
- net ClampL: track 0.00 -> 12.7 mm
- net GNDPWR: track 0.00 -> 2.54 mm
- net ClampH: track 0.80 -> 0.00 mm
- net OutH2: vias 0 -> 12
- added copper zone on F.Cu, net ClampL
- added copper zone on B.Cu, net GNDPWR
- added copper zone on F.Cu, net GNDPWR
- added copper zone on B.Cu, net OutH2
- added copper zone on F.Cu, net OutH2
- added copper zone on F.Cu, net OutL2
- removed copper zone on B.Cu, net Drain_Low
- removed copper zone on F.Cu, net Drain_Low
- removed copper zone on B.Cu, net VDC
- removed copper zone on F.Cu, net VDC
Other:
- board size 114.4 x 54.6 mm -> 67.7 x 59.6 mm
