File: Driver_Test.kicad_pcb (KiCad board)
At the start: 2 copper layers, 67.7 x 39.7 mm, 20 parts, among them J1 Conn_02x05_Odd_Even, J2 Conn_02x05_Odd_Even, J3 Conn_02x16_Odd_Even

Commit message: VER1.0.2: сделал плату на один ключ
Parts:
- removed D1: ~, Mornsun:QAxCx
- removed D2: NSI6651, Package_SO:SOIC-16W_7.5x10.3mm_P1.27mm
- removed D8: ~, Mornsun:K78xxM-1000R3
- removed J3: Conn_02x16_Odd_Even, Connector_PinSocket_2.00mm:PinSocket_2x16_P2.00mm_Vertical
- added C11: 4.7u, Capacitor_SMD:C_1206_3216Metric_Pad1.33x1.80mm_HandSolder, F.Cu at (7.25, 1.18)
- added C12: 4.7u, Capacitor_SMD:C_1206_3216Metric_Pad1.33x1.80mm_HandSolder, F.Cu at (7.25, 4.53)
- added C13: 100p, Capacitor_SMD:C_1206_3216Metric_Pad1.33x1.80mm_HandSolder, F.Cu at (7.25, 7.88)
- added C25: 56p, Capacitor_SMD:C_0805_2012Metric_Pad1.18x1.45mm_HandSolder, F.Cu at (6.66, 11.1)
- added C26: 56p, Capacitor_SMD:C_0805_2012Metric_Pad1.18x1.45mm_HandSolder, F.Cu at (6.66, 14.1)
- added D16: ~, LED_SMD:LED_0805_2012Metric_Pad1.15x1.40mm_HandSolder, F.Cu at (12.7, 1.02)
- added D17: ~, LED_SMD:LED_0805_2012Metric_Pad1.15x1.40mm_HandSolder, F.Cu at (12.7, 4.06)
- added L2: 22u, Inductor_SMD:L_1812_4532Metric_Pad1.30x3.40mm_HandSolder, F.Cu at (7.91, 18.0)
- added Q1: ~, Package_TO_SOT_SMD:SOT-23, F.Cu at (11.5, 11.9)
- added R10: 10k, Resistor_SMD:R_0805_2012Metric_Pad1.20x1.40mm_HandSolder, F.Cu at (1.88, 12.8)
- added R11: 1k, Resistor_SMD:R_0805_2012Metric_Pad1.20x1.40mm_HandSolder, F.Cu at (1.88, 15.7)
- added R12: 560, Resistor_SMD:R_0805_2012Metric_Pad1.20x1.40mm_HandSolder, F.Cu at (1.88, 18.7)
- added R13: 4.7k, Resistor_SMD:R_0805_2012Metric_Pad1.20x1.40mm_HandSolder, F.Cu at (1.88, 21.6)
- added R3: 0, Resistor_SMD:R_0805_2012Metric_Pad1.20x1.40mm_HandSolder, F.Cu at (1.88, 0.97)
- added R4: 0, Resistor_SMD:R_0805_2012Metric_Pad1.20x1.40mm_HandSolder, F.Cu at (1.88, 3.92)
- added R8: 1k, Resistor_SMD:R_0805_2012Metric_Pad1.20x1.40mm_HandSolder, F.Cu at (1.88, 6.88)
- added R9: 1k, Resistor_SMD:R_0805_2012Metric_Pad1.20x1.40mm_HandSolder, F.Cu at (1.88, 9.82)
- D7: moved to F.Cu
- J2: value Conn_02x05_Odd_Even -> Conn_02x02_Odd_Even; footprint Connector_PinHeader_2.54mm:PinHeader_2x05_P2.54mm_Horizontal -> Connector_PinHeader_2.54mm:PinHeader_2x02_P2.54mm_Horizontal
- moved J2 33.0 mm to (335.7, 307.3)
- moved D7 10.0 mm to (334.8, 294.8), turned to -90 degrees
- moved D9 3.50 mm to (323.5, 294.8)
Connections:
- J2 pad 1: GNDPWR -> unconnected-(J2-Pin_1-Pad1)
- J2 pad 2: GNDPWR -> unconnected-(J2-Pin_2-Pad2)
- J2 pad 3: OutH2 -> unconnected-(J2-Pin_3-Pad3)
- J2 pad 4: OutH2 -> unconnected-(J2-Pin_4-Pad4)
Other:
- board size 67.7 x 39.7 mm -> 25.7 x 39.8 mm

Commit message: VER1.0.2: обновил модель платы драйверов
Parts:
- removed C13: 100p, Capacitor_SMD:C_1206_3216Metric_Pad1.33x1.80mm_HandSolder
- removed C18: 0.1u, Capacitor_SMD:C_0805_2012Metric_Pad1.18x1.45mm_HandSolder
- removed D12: D_Zener_Small, Diode_SMD:D_SOD-323_HandSoldering
- removed Q1: ~, Package_TO_SOT_SMD:SOT-23
- removed R13: 4.7k, Resistor_SMD:R_0805_2012Metric_Pad1.20x1.40mm_HandSolder
- removed R3, R4: 0, Resistor_SMD:R_0805_2012Metric_Pad1.20x1.40mm_HandSolder
- removed R8: 1k, Resistor_SMD:R_0805_2012Metric_Pad1.20x1.40mm_HandSolder
- added J3: Conn_02x05_Odd_Even, Connector_PinSocket_2.54mm:PinSocket_2x05_P2.54mm_Vertical, F.Cu at (324.0, 279.5)
- added L1: 12u, Inductor_SMD:L_1210_3225Metric_Pad1.42x2.65mm_HandSolder, B.Cu at (330.0, 292.2)
- added R1: 510, Resistor_SMD:R_0805_2012Metric_Pad1.20x1.40mm_HandSolder, F.Cu at (321.5, 315.2)
- added R5: 698, Resistor_SMD:R_0805_2012Metric_Pad1.20x1.40mm_HandSolder, F.Cu at (319.2, 304.2)
- added R6: 1k, Resistor_SMD:R_0805_2012Metric_Pad1.20x1.40mm_HandSolder, F.Cu at (317.5, 307.5)
- C11, C12, C25, C26, D13, R11, R12: moved to B.Cu
- C15, C22: value 0.1u -> 10u
- C19: value 1u -> 2.2u
- D10: footprint Diode_SMD:D_SMB_Handsoldering -> Diode_SMD:D_SMA_Handsoldering
- L2: value 22u -> 47u; moved to B.Cu
- moved C11 438.4 mm to (331.8, 296.0)
- moved C12 434.8 mm to (333.2, 292.2), turned to -90 degrees
- moved R9 423.4 mm to (322.8, 286.0), turned to 90 degrees
- moved L2 420.9 mm to (331.5, 287.2)
- moved R10 419.9 mm to (320.8, 286.0), turned to 90 degrees
- moved C25 418.9 mm to (322.8, 286.0), turned to 90 degrees
- moved C26 415.5 mm to (320.8, 286.0), turned to 90 degrees
- moved D16 414.6 mm to (319.0, 280.5)
- moved D17 414.1 mm to (319.0, 282.8)
- moved R11 413.1 mm to (319.0, 280.5), turned to 180 degrees
- moved R12 412.7 mm to (319.0, 282.8), turned to 180 degrees
- moved D10 10.2 mm to (337.0, 316.5), turned to -90 degrees
- moved C15 6.31 mm to (321.2, 300.2), turned to 180 degrees
- moved C22 6.31 mm to (326.5, 300.2), turned to 180 degrees
- moved C14 5.46 mm to (321.2, 302.8), turned to 180 degrees
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Connections:
- C12 pad 1: Net-(D7-Vin) -> Net-(C12-Pad1)
- D9 pad 4: OutH2 -> OutGate
- D9 pad 6: OutL2 -> OutGate
- J1 pad 1: GNDPWR -> ClampL
- J1 pad 10: OUT -> ClampL
- J1 pad 2: GNDPWR -> ClampL
- J1 pad 3: OutH2 -> GNDPWR
- J1 pad 4: OutH2 -> GNDPWR
- J1 pad 5: OutL2 -> OutGate
- J1 pad 6: OutL2 -> OutGate
- J1 pad 7: ClampL -> GNDPWR
- J1 pad 8: ClampL -> GNDPWR
- J1 pad 9: OUT -> ClampL
- J2 pad 3: unconnected-(J2-Pin_3-Pad3) -> OUT
- J2 pad 4: unconnected-(J2-Pin_4-Pad4) -> OUT
- L2 pad 1: +15V -> Net-(C12-Pad1)
- R2 pad 1: Net-(D12-K) -> Net-(D11-A)
- R2 pad 2: Net-(D13-K) -> Net-(R1-Pad1)
Routing:
- net ClampL: track 0.00 -> 28.7 mm
- net Net-(R1-Pad1): track 0.00 -> 16.1 mm
- net Net-(D13-K): track 0.00 -> 9.49 mm, vias 0 -> 1
- net GNDPWR: track 0.00 -> 5.05 mm
- net OUT: track 0.00 -> 4.62 mm
- net ~{FLT}: track 0.00 -> 4.61 mm, vias 0 -> 1
- net RDY: track 0.00 -> 4.61 mm, vias 0 -> 1
- net Net-(D11-A): track 0.00 -> 4.25 mm
- net Net-(D10-A): track 0.00 -> 4.25 mm
- net -15VL: track 0.00 -> 2.69 mm, vias 0 -> 2
- net Net-(D16-A): track 0.00 -> 2.02 mm, vias 0 -> 1
- net Net-(D17-A): track 0.00 -> 1.98 mm, vias 0 -> 1
- net +15VL: track 0.00 -> 1.26 mm, vias 0 -> 1
- added copper zone on B.Cu, net GNDPWR
- added copper zone on F.Cu, net OutGate
Other:
- board size 25.7 x 39.8 mm -> 25.7 x 44.8 mm
- copper layers 2 -> 4

Commit message: VER1.0.2: развел все дорожки, добавил светодиоды по питанию
Parts:
- removed R5: 698, Resistor_SMD:R_0805_2012Metric_Pad1.20x1.40mm_HandSolder
- removed R6: 1k, Resistor_SMD:R_0805_2012Metric_Pad1.20x1.40mm_HandSolder
- added D1: ~, Diode_SMD:D_SOD-323_HandSoldering, F.Cu at (317.5, 316.2)
- added D2: ~, LED_SMD:LED_0805_2012Metric_Pad1.15x1.40mm_HandSolder, F.Cu at (338.0, 280.5)
- added D3: ~, LED_SMD:LED_0805_2012Metric_Pad1.15x1.40mm_HandSolder, F.Cu at (338.0, 282.8)
- added R3: 1k, Resistor_SMD:R_0805_2012Metric_Pad1.20x1.40mm_HandSolder, B.Cu at (338.0, 280.5)
- added R4: 3k, Resistor_SMD:R_0805_2012Metric_Pad1.20x1.40mm_HandSolder, B.Cu at (338.0, 282.8)
- moved C11 9.49 mm to (328.8, 287.0), turned to -90 degrees
- moved R2 9.22 mm to (317.5, 311.2), turned to 90 degrees
- moved L1 7.20 mm to (332.5, 285.5), turned to 0 degrees
- moved L2 5.77 mm to (332.0, 293.0), turned to -90 degrees
- moved R10 3.88 mm to (324.5, 285.0), turned to 0 degrees
- moved C12 3.82 mm to (332.5, 288.5), turned to 180 degrees
- moved R12 3.20 mm to (321.0, 285.2), turned to -90 degrees
- moved C26 3.01 mm to (318.8, 288.2), turned to 180 degrees
- moved C25 2.06 mm to (324.8, 285.5), turned to 0 degrees
- moved R9 2.02 mm to (324.5, 287.0), turned to 0 degrees
- moved R1 1.52 mm to (321.2, 313.8), turned to 0 degrees
- moved R11 1.25 mm to (319.0, 281.8), turned to -90 degrees
Connections:
- C11 pad 2: GND1 -> GND
- C12 pad 2: GND1 -> GND
- D11 pad 2: Net-(D11-A) -> Net-(D1-A)
- D7 pad 2: GND1 -> GND
- J2 pad 2: unconnected-(J2-Pin_2-Pad2) -> OUT
- J2 pad 3: OUT -> unconnected-(J2-Pin_3-Pad3)
- J3 pad 1: GND1 -> GND
- R1 pad 1: Net-(R1-Pad1) -> Net-(D13-K)
- R2 pad 1: Net-(D11-A) -> Net-(D1-K)
- R2 pad 2: Net-(R1-Pad1) -> Net-(D13-K)
Routing:
- net +15VL: track 1.26 -> 24.3 mm, vias 1 -> 2
- net GND: track 0.00 -> 19.1 mm, vias 0 -> 6
- net Net-(R1-Pad1): track 16.1 -> 0.00 mm
- net -15VL: track 2.69 -> 18.6 mm
- net ~{FLT}: track 4.61 -> 20.3 mm, vias 1 -> 2
- net PWM_N: track 0.00 -> 14.9 mm, vias 0 -> 1
- net RST: track 0.00 -> 14.8 mm, vias 0 -> 1
- net PWM_P: track 0.00 -> 13.8 mm, vias 0 -> 1
- net Net-(D7-Vin): track 0.00 -> 13.7 mm
- net Net-(D1-A): track 0.00 -> 11.2 mm
- net Net-(D13-K): track 9.49 -> 18.8 mm
- net Net-(C12-Pad1): track 0.00 -> 6.16 mm
- net +5V: track 0.00 -> 5.76 mm, vias 0 -> 1
- net GNDPWR: track 5.05 -> 10.3 mm, vias 0 -> 1
- net RDY: track 4.61 -> 8.96 mm
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- added copper zone on B.Cu, net +15V
- added copper zone on In2.Cu, net +15VL
- added copper zone on F.Cu, net +5V
- added copper zone on B.Cu, net -15VL
- added copper zone on In1.Cu, net GND
- added copper zone on In1.Cu, net GNDPWR
Other:
- board text added: "+15V"
- board text added: "+5V"
- board text added: "CL"
- board text added: "D"
- board text added: "G"
- board text added: "S"
