File: Driver_Test.kicad_sch (KiCad schematic)
At the start: 62 parts, among them J1 Conn_02x05_Odd_Even, J2 Conn_02x05_Odd_Even, J3 Conn_02x16_Odd_Even

Commit message: VER1.0.2: сделал плату на один ключ
Parts:
- removed C1, C9: 10u, Capacitor_SMD:C_1206_3216Metric_Pad1.33x1.80mm_HandSolder, symbol Device:C_Small
- removed C10, C2: 0.1u, Capacitor_SMD:C_1206_3216Metric_Pad1.33x1.80mm_HandSolder, symbol Device:C_Small
- removed C16, C17: 10u, Capacitor_SMD:C_1210_3225Metric_Pad1.33x2.70mm_HandSolder, symbol Device:C_Small
- removed C23, C24: 2.2u, Capacitor_SMD:C_0805_2012Metric_Pad1.18x1.45mm_HandSolder, symbol Device:C_Small
- removed C3, C4: 4.7u, Capacitor_SMD:C_1206_3216Metric_Pad1.33x1.80mm_HandSolder, symbol Device:C_Small
- removed C5: 100p, Capacitor_SMD:C_1206_3216Metric_Pad1.33x1.80mm_HandSolder, symbol Device:C_Small
- removed C6: 0.1u, Capacitor_SMD:C_0805_2012Metric_Pad1.18x1.45mm_HandSolder, symbol Device:C_Small
- removed C7: 1u, Capacitor_SMD:C_0805_2012Metric_Pad1.18x1.45mm_HandSolder, symbol Device:C_Small
- removed C8: 100p, Capacitor_SMD:C_0805_2012Metric_Pad1.18x1.45mm_HandSolder, symbol Device:C_Small
- removed D1: ~, QAxCx, symbol Mornsun:QAxCx
- removed D14: ~, Package_SO:SOIC-8_3.9x4.9mm_P1.27mm, symbol Interface_My:ADM3485E
- removed D15: ~, Package_TO_SOT_SMD:SOT-23-5, symbol Logic_My:SN74AHC1G08DBVR
- removed D2: NSI6651, Package_SO:SOIC-16W_7.5x10.3mm_P1.27mm, symbol Driver_My:NSI6651
- removed D3, D4: D_Small, Diode_SMD:D_SMB_Handsoldering, symbol Device:D_Small
- removed D5: D_Zener_Small, Diode_SMD:D_SOD-323_HandSoldering, symbol Device:D_Zener_Small
- removed D6: ~, Diode_SMD:D_SOD-123, symbol Device:D_Schottky_Small
- removed D8: ~, Mornsun:K78xxM-1000R3, symbol Mornsun:K78xxM-1000R3 ÕýÊä³ö
- removed J2: Conn_02x05_Odd_Even, Connector_PinHeader_2.54mm:PinHeader_2x05_P2.54mm_Horizontal, symbol Connector_Generic:Conn_02x05_Odd_Even
- removed J3: Conn_02x16_Odd_Even, Connector_PinSocket_2.00mm:PinSocket_2x16_P2.00mm_Vertical, symbol Connector_Generic:Conn_02x16_Odd_Even
- removed L1: 22u, Inductor_SMD:L_1812_4532Metric_Pad1.30x3.40mm_HandSolder, symbol Device:L_Small
- removed R1: Rdesat, Resistor_SMD:R_0805_2012Metric_Pad1.20x1.40mm_HandSolder, symbol Device:R_Small
- removed R5, R6: 0, Resistor_SMD:R_0805_2012Metric_Pad1.20x1.40mm_HandSolder, symbol Device:R_Small
- removed R7: 120, Resistor_SMD:R_0805_2012Metric_Pad1.20x1.40mm_HandSolder, symbol Device:R_Small
- added J2: Conn_02x02_Odd_Even, Connector_PinHeader_2.54mm:PinHeader_2x02_P2.54mm_Horizontal, symbol Connector_Generic:Conn_02x02_Odd_Even
Connections:
- no-connect marks 1 -> 0
Other:
- note removed: "Автоматический RST"
- note removed: "Драйвер верхнего ключа"
- note removed: "Питание 5В"
- note removed: "Питание верхнего драйвера"

Commit message: VER1.0.2: обновил модель платы драйверов
Parts:
- removed C13: 100p, Capacitor_SMD:C_1206_3216Metric_Pad1.33x1.80mm_HandSolder, symbol Device:C_Small
- removed C18: 0.1u, Capacitor_SMD:C_0805_2012Metric_Pad1.18x1.45mm_HandSolder, symbol Device:C_Small
- removed D12: D_Zener_Small, Diode_SMD:D_SOD-323_HandSoldering, symbol Device:D_Zener_Small
- removed Q1: ~, Package_TO_SOT_SMD:SOT-23, symbol Transistor_FET:2N7002
- removed R13: 4.7k, Resistor_SMD:R_0805_2012Metric_Pad1.20x1.40mm_HandSolder, symbol Device:R_Small
- removed R3, R4: 0, Resistor_SMD:R_0805_2012Metric_Pad1.20x1.40mm_HandSolder, symbol Device:R_Small
- removed R8: 1k, Resistor_SMD:R_0805_2012Metric_Pad1.20x1.40mm_HandSolder, symbol Device:R_Small
- added J3: Conn_02x05_Odd_Even, Connector_PinSocket_2.54mm:PinSocket_2x05_P2.54mm_Vertical, symbol Connector_Generic:Conn_02x05_Odd_Even
- added L2: 47u, Inductor_SMD:L_1812_4532Metric_Pad1.30x3.40mm_HandSolder, symbol Device:L_Small
- added R1: 510, Resistor_SMD:R_0805_2012Metric_Pad1.20x1.40mm_HandSolder, symbol Device:R_Small
- added R5: 698, Resistor_SMD:R_0805_2012Metric_Pad1.20x1.40mm_HandSolder, symbol Device:R_Small
- added R6: 1k, Resistor_SMD:R_0805_2012Metric_Pad1.20x1.40mm_HandSolder, symbol Device:R_Small
- C15, C22: value 0.1u -> 10u
- C19: value 1u -> 2.2u
- D10: footprint Diode_SMD:D_SMB_Handsoldering -> Diode_SMD:D_SMA_Handsoldering
- L1: renamed from L2; value 22u -> 12u; footprint Inductor_SMD:L_1812_4532Metric_Pad1.30x3.40mm_HandSolder -> Inductor_SMD:L_1210_3225Metric_Pad1.42x2.65mm_HandSolder
Connections:
- net +15V: now also J3.2 (Pin_2)
- net +15VL: now also R1.2
- net +5V: now also J3.4 (Pin_4)
- net ClampL: now also J1.1 (Pin_1), J1.10 (Pin_10), J1.2 (Pin_2), J1.9 (Pin_9); no longer J1.7 (Pin_7), J1.8 (Pin_8)
- net GND: now also J3.3 (Pin_3), J3.5 (Pin_5), J3.7 (Pin_7), J3.9 (Pin_9)
- net GND1: now also J3.1 (Pin_1)
- net GNDPWR: now also J1.3 (Pin_3), J1.4 (Pin_4), J1.7 (Pin_7), J1.8 (Pin_8), R5.1; no longer J1.1 (Pin_1), J1.2 (Pin_2)
- net OUT: now also J2.3 (Pin_3), J2.4 (Pin_4); no longer J1.10 (Pin_10), J1.9 (Pin_9)
- net PWM_N: now also J3.10 (Pin_10)
- net PWM_P: now also J3.8 (Pin_8)
- net RST: now also J3.6 (Pin_6)
- net at C12.1, L1.2: now also L2.1; no longer D7.1 (Vin)
- net at C20.2, D13.1 (K), D9.2 (DESAT): now also R5.2, R6.1; no longer R2.2
- net at R2.1: now also D11.2 (A)
- removed net OutH2: D9.4 (OUTH), J1.3 (Pin_3), J1.4 (Pin_4)
- net OutL2 renamed OutGate
- net OutGate: now also D9.4 (OUTH)
- new net: D7.1 (Vin), L2.2
- new net: R1.1, R2.2, R6.2
- no-connect marks 0 -> 2
Other:
- note removed: "Защита от одновременного включения"
- note removed: "Опции RESET"
- note removed: "Сброс ошибки драйвера"
- moved on the sheet: C19, C20, D10, D11, D13, R2

Commit message: VER1.0.2: развел все дорожки, добавил светодиоды по питанию
Parts:
- removed R5: 698, Resistor_SMD:R_0805_2012Metric_Pad1.20x1.40mm_HandSolder, symbol Device:R_Small
- removed R6: 1k, Resistor_SMD:R_0805_2012Metric_Pad1.20x1.40mm_HandSolder, symbol Device:R_Small
- added D1: ~, Diode_SMD:D_SOD-323_HandSoldering, symbol Device:D_Schottky_Small
- added D2, D3: ~, LED_SMD:LED_0805_2012Metric_Pad1.15x1.40mm_HandSolder, symbol Device:LED_Small
- added R3: 1k, Resistor_SMD:R_0805_2012Metric_Pad1.20x1.40mm_HandSolder, symbol Device:R_Small
- added R4: 3k, Resistor_SMD:R_0805_2012Metric_Pad1.20x1.40mm_HandSolder, symbol Device:R_Small
Connections:
- net GND1 is gone; now on net GND: C11.2, C12.2, D7.2 (GND), J3.1 (Pin_1)
- net +15V: now also D3.2 (A)
- net +5V: now also D2.2 (A)
- net GND: now also R3.1, R4.1
- net OUT: now also J2.2 (Pin_2); no longer J2.3 (Pin_3)
- net at C20.2, D13.1 (K), D9.2 (DESAT): now also R1.1, R2.2
- net at R2.1: now also D1.1 (K); no longer D11.2 (A)
- new net: D3.1 (K), R4.2
- new net: D2.1 (K), R3.2
- new net: D1.2 (A), D11.2 (A)
Other:
- moved on the sheet: R1, R2
